File: KiCad/LaunchController/Interface.kicad_sch (KiCad schematic)
At the start: 158 parts

Commit message: 修正を回路図に反映
Parts:
- removed C? (x10): 0.1uF, Capacitor_SMD:C_0603_1608Metric_Pad1.08x0.95mm_HandSolder, symbol Device:C_Small
- removed J?: JMP_VALVE_CLOSE, Connector_PinHeader_2.54mm:PinHeader_1x02_P2.54mm_Vertical, symbol Connector:Conn_01x02_Pin
- removed J?: JMP_PURGE, Connector_PinHeader_2.54mm:PinHeader_1x02_P2.54mm_Vertical, symbol Connector:Conn_01x02_Pin
- removed J?: JMP_SAFETY, Connector_PinHeader_2.54mm:PinHeader_1x02_P2.54mm_Vertical, symbol Connector:Conn_01x02_Pin
- removed J?: JMP_EMERGENCY_STOP, Connector_PinHeader_2.54mm:PinHeader_1x02_P2.54mm_Vertical, symbol Connector:Conn_01x02_Pin
- removed J?: JMP_IGNITOR, Connector_PinHeader_2.54mm:PinHeader_1x02_P2.54mm_Vertical, symbol Connector:Conn_01x02_Pin
- removed J?: JMP_FILL, Connector_PinHeader_2.54mm:PinHeader_1x02_P2.54mm_Vertical, symbol Connector:Conn_01x02_Pin
- removed J?: JMP_SEQUENCE_START, Connector_PinHeader_2.54mm:PinHeader_1x02_P2.54mm_Vertical, symbol Connector:Conn_01x02_Pin
- removed J?: JMP_DUMP, Connector_PinHeader_2.54mm:PinHeader_1x02_P2.54mm_Vertical, symbol Connector:Conn_01x02_Pin
- removed J?: JMP_VALVE_OPEN, Connector_PinHeader_2.54mm:PinHeader_1x02_P2.54mm_Vertical, symbol Connector:Conn_01x02_Pin
- removed J?: JMP_O2, Connector_PinHeader_2.54mm:PinHeader_1x02_P2.54mm_Vertical, symbol Connector:Conn_01x02_Pin
- removed Q? (x11): 2SC3325-Y, Package_TO_SOT_SMD:SC-59_Handsoldering, symbol Device:Q_NPN_BEC
- removed R? (x31): 10kR, Resistor_SMD:R_0603_1608Metric_Pad0.98x0.95mm_HandSolder, symbol Device:R_Small
- removed R? (x11): 270R, Resistor_SMD:R_0603_1608Metric_Pad0.98x0.95mm_HandSolder, symbol Device:R_Small
- removed R? (x11): 2kR, Resistor_SMD:R_0603_1608Metric_Pad0.98x0.95mm_HandSolder, symbol Device:R_Small
- added C17 (x3): 0.1uF, Capacitor_SMD:C_0603_1608Metric_Pad1.08x0.95mm_HandSolder, symbol Device:C_Small
- added D? (x3): LED, LED_SMD:LED_0603_1608Metric_Pad1.05x0.95mm_HandSolder, symbol Device:LED_Small
- added R16, R19, R? (x9): 1kR, Resistor_SMD:R_0603_1608Metric_Pad0.98x0.95mm_HandSolder, symbol Device:R_Small
- added U5, U? (x5): U74HC14, Package_DIP:DIP-14_W7.62mm, symbol 74xx:74HC14
Connections:
- net LED_CONFIRM is gone; now on net CONN_LED_CONFIRM: R?.1
- net LED_DUMP is gone; now on net CONN_LED_DUMP: R?.1
- net LED_FILL is gone; now on net CONN_LED_FILL: R?.1
- net LED_IGNITOR is gone; now on net CONN_LED_IGNITOR: R?.1
- net LED_O2 is gone; now on net CONN_LED_O2: R?.1
- net LED_POWER is gone; now on net CONN_LED_POWER: R?.1
- net LED_PURGE is gone; now on net CONN_LED_PURGE: R?.1
- net LED_SAFTEY is gone; now on net CONN_LED_SAFTEY: R?.1
- net LED_SEQUENCE is gone; now on net CONN_LED_SEQUENCE: R?.1
- net LED_VALVE_CLOSE is gone; now on net CONN_LED_VALVE_CLOSE: R?.1
- net LED_VALVE_OPEN is gone; now on net CONN_LED_VALVE_OPEN: R?.1
- net +5V: now also C17.2, C17.2, C17.2, U?.14 (VCC)
- net GND: now also C17.1, C17.1, C17.1, D?.1 (K), D?.1 (K), D?.1 (K), U?.7 (GND)
- net SW_DUMP: now also R?.1
- net SW_EMERGENCY_STOP: now also R?.1
- net SW_FILL: now also R?.1
- net SW_IGNITOR: now also R?.1
- net SW_KILL: now also R16.1
- net SW_O2: now also R?.1
- net SW_PURGE: now also R?.1
- net SW_RESET: now also R19.1
- net SW_SAFETY: now also R?.1
- net SW_SEQUENCE_START: now also R?.1
- net SW_VALVE_CLOSE: now also R?.1
- net SW_VALVE_OPEN: now also R?.1
- new net: D?.2 (A), R?.2 (x3)
- new net: R?.2, U?.3 (x4)
- new net: R16.2, U5.1
- new net: R19.2, U5.3
- new net CONN_LED_ERROR: R?.2
- new net CONN_LED_LOW_VOLTAGE: R?.2
- new net CONN_LED_SHIFT: R?.1
- new net CTL_CONFIRM_1: U?.4
- new net CTL_CONFIRM_2: U?.4
- new net CTL_CONFIRM_3: U?.4
- new net CTL_KILL: U5.2
- new net CTL_RESET: U5.4
- new net CTL_SHIFT: U?.4
- new net LED_ERROR: R?.1, R?.1
- new net LED_LOW_VOLTAGE: R?.1, R?.1
- new net SW_CONFIRM_1: R?.1
- new net SW_CONFIRM_2: R?.1
- new net SW_CONFIRM_3: R?.1
- new net SW_SHIFT: R?.1
Other:
- note added: "CONFIRM 1 SWITCH A ALT PU"
- note added: "CONFIRM 2 SWITCH A ALT PU"
- note added: "CONFIRM 3 SWITCH A ALT PU"
- note added: "DUMP SWITCH A ALT PU"
- note added: "EMERGENCY STOP SWITCH A ALT PU"
- note added: "FILL SWITCH A MOM PU"
- note added: "IGNITOR SWITCH A ALT PU"
- note added: "KILL SWITCH A MOMENTARY PU"
- note added: "LED_COM"
- note added: "LED_ERROR"
- note added: "LED_LOW_VOLTAGE"
- note added: "LED_SHIFT"
- note added: "LED_TASK"
- note added: "O2 SWITCH A ALT PU"
- note added: "PURGE SWITCH A ALT PU"
- note added: "RESET SWITCH A MOMENTARY PD"
- note added: "SAFETY SWITCH A ALT PU"
- note added: "SEQUENCE START SWITCH A MOM PU"
- note added: "SHIFT SWITCH A ALT PU"
- note added: "VALVE CLOSE SWITCH A ALT PU"
- note added: "VALVE OPEN SWITCH A ALT PU"
- note removed: "DUMP SWITCH A ALTERNAIT"
- note removed: "EMERGENCY STOP SWITCH A ALTERNAIT"
- note removed: "FILL SWITCH A MOMENTARY"
- note removed: "IGNITOR SWITCH A ALTERNAIT"
- note removed: "LED_PING"
- note removed: "LED_STATUS"
- note removed: "O2 SWITCH A ALTERNAIT"
- note removed: "PURGE SWITCH A ALTERNAIT"
- note removed: "SAFETY SWITCH A ALTERNAIT"
- note removed: "SEQUENCE START SWITCH A MOMENTARY"
- note removed: "VALVE CLOSE SWITCH A ALTERNAIT"
- note removed: "VALVE OPEN SWITCH A ALTERNAIT"
- moved on the sheet: D?, J?, R?, U?A, U?B, U?C, U?D, U?E, U?F, U?G

Commit message: フィードバックLEDを追加
Parts:
- removed R? (x6): 1kR, Resistor_SMD:R_0603_1608Metric_Pad0.98x0.95mm_HandSolder, symbol Device:R_Small
- removed U? (x6): U74HC14, Package_DIP:DIP-14_W7.62mm, symbol 74xx:74HC14
- added D? (x8): LED, LED_SMD:LED_0603_1608Metric_Pad1.05x0.95mm_HandSolder, symbol Device:LED_Small
- added J2: JMP_RUN, Connector_PinHeader_2.54mm:PinHeader_1x02_P2.54mm_Vertical, symbol Connector:Conn_01x02_Pin
- added R? (x14): 1kR, Resistor_SMD:R_0603_1608Metric_Pad0.98x0.95mm_HandSolder, symbol Device:R_Small
- added U? (x6): U74HC14, Package_DIP:DIP-14_W7.62mm, symbol 74xx:74HC14
Connections:
- net CTL_CONFIRM_1: now also U?.4
- net CTL_CONFIRM_2: now also U?.4
- net CTL_CONFIRM_3: now also U?.4
- net CTL_EMERGENCY_STOP: now also U?.8
- net CTL_SAFETY: now also U?.6
- net CTL_SEQUENCE_START: now also U?.10
- net GND: now also D?.1 (K), D?.1 (K), D?.1 (K), D?.1 (K), D?.1 (K), D?.1 (K), D?.1 (K), D?.1 (K), J2.1 (Pin_1)
- net SW_CONFIRM_1: now also R?.1
- net SW_CONFIRM_2: now also R?.1
- net SW_CONFIRM_3: now also R?.1
- net SW_EMERGENCY_STOP: now also R?.1
- net SW_SAFETY: now also R?.1
- net SW_SEQUENCE_START: now also R?.1
- net CONN_LED_CONFIRM renamed CONN_LED_EMERGENCY
- net CONN_LED_VALVE_CLOSE renamed CONN_LED_CLOSE
- net CONN_LED_VALVE_OPEN renamed CONN_LED_OPEN
- net CTL_VALVE_CLOSE renamed CTL_CLOSE
- net CTL_VALVE_OPEN renamed CTL_OPEN
- net SW_VALVE_CLOSE renamed SW_CLOSE
- net SW_VALVE_OPEN renamed SW_OPEN
- new net: R?.2, U?.9
- new net: R?.2, U?.3 (x3)
- new net: D?.2 (A), R?.2 (x8)
- new net: R?.2, U?.11
- new net: R?.2, U?.5
- new net CONN_FB_LED_O2: R?.1
- new net CONN_LED_FB_CLOSE: R?.1
- new net CONN_LED_FB_DUMP: R?.1
- new net CONN_LED_FB_FILL: R?.1
- new net CONN_LED_FB_IGNITOR: R?.1
- new net CONN_LED_FB_OPEN: R?.1
- new net CONN_LED_FB_PURGE: R?.1
- new net CONN_LED_FB_SHIFT: R?.1
- new net CTL_RUN: J2.2 (Pin_2)
Other:
- note added: "CLOSE SWITCH A ALT PU"
- note added: "LED_CLOSE"
- note added: "LED_EMERGENCY"
- note added: "LED_FB_CLOSE"
- note added: "LED_FB_DUMP"
- note added: "LED_FB_FILL"
- note added: "LED_FB_IGNITOR"
- note added: "LED_FB_O2"
- note added: "LED_FB_OPEN"
- note added: "LED_FB_PURGE"
- note added: "LED_FB_SHIFT"
- note added: "LED_OPEN"
- note added: "OPEN SWITCH A ALT PU"
- note added: "RUN SWITCH A MOMENTARY"
- note removed: "LED_CONFIRM"
- note removed: "LED_VALVE_CLOSE"
- note removed: "LED_VALVE_OPEN"
- note removed: "VALVE CLOSE SWITCH A ALT PU"
- note removed: "VALVE OPEN SWITCH A ALT PU"
- moved on the sheet: C17, D?, J?, R?, U?A, U?B, U?C, U?D, U?E, U?F, U?G
