File: KiCad/LaunchController/Indicator.kicad_sch (KiCad schematic)
At the start: 46 parts

Commit message: ランコンおわり
Parts:
- removed D?: LED, LED_SMD:LED_0603_1608Metric_Pad1.05x0.95mm_HandSolder, symbol Device:LED_Small
- removed R?: 1kR, Resistor_SMD:R_0603_1608Metric_Pad0.98x0.95mm_HandSolder, symbol Device:R_Small
Other:
- note removed: "LED_POWER"
Changed lines of the file:
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@@
   (junction (at 63.5 101.6) (diameter 0) (color 0 0 0 0)
   )
-  (junction (at 156.21 38.1) (diameter 0) (color 0 0 0 0)
-  )
   (junction (at 20.32 38.1) (diameter 0) (color 0 0 0 0)
   )
@@
     (stroke (width 0) (type default))
   )
-  (wire (pts (xy 161.29 38.1) (xy 156.21 38.1))
-    (stroke (width 0) (type default))
-  )
   (wire (pts (xy 85.09 104.14) (xy 85.09 101.6))
     (stroke (width 0) (type default))
@@
     (stroke (width 0) (type default))
   )
-  (wire (pts (xy 156.21 40.64) (xy 156.21 38.1))
-    (stroke (width 0) (type default))
-  )
   (wire (pts (xy 68.58 38.1) (xy 63.5 38.1))
     (stroke (width 0) (type default))
@@
     (stroke (width 0) (type default))
   )
-  (wire (pts (xy 161.29 55.88) (xy 161.29 53.34))
-    (stroke (width 0) (type default))
-  )
   (wire (pts (xy 209.55 45.72) (xy 209.55 48.26))
     (stroke (width 0) (type default))
@@
     (stroke (width 0) (type default))
   )
-  (wire (pts (xy 161.29 45.72) (xy 161.29 48.26))
-    (stroke (width 0) (type default))
-  )
   (wire (pts (xy 269.24 40.64) (xy 269.24 38.1))
     (stroke (width 0) (type default))
@@
     (stroke (width 0) (type default))
   )
-  (wire (pts (xy 161.29 40.64) (xy 161.29 38.1))
-    (stroke (width 0) (type default))
-  )
   (wire (pts (xy 38.1 173.99) (xy 40.64 173.99))
     (stroke (width 0) (type default))
@@
     (stroke (width 0) (type default))
   )
-  (wire (pts (xy 156.21 35.56) (xy 156.21 38.1))
+  (wire (pts (xy 38.1 143.51) (xy 40.64 143.51))
     (stroke (width 0) (type default))
   )
@@
   )
   (rectangle (start 218.44 76.2) (end 238.76 138.43)
-    (stroke (width 0) (type default))
-    (fill (type none))
-  )
-  (rectangle (start 148.59 12.7) (end 168.91 74.93)
     (stroke (width 0) (type default))
     (fill (type none))
@@
     (effects (font (size 1.27 1.27)) (justify left bottom))
   )
-  (text "LED_POWER\n" (at 149.86 15.24 0)
-    (effects (font (size 1.27 1.27)) (justify left bottom))
-  )
   (global_label "CONN_LED_FB_DUMP" (shape output) (at 40.64 173.99 0) (fields_autoplaced)
     (effects (font (size 1.27 1.27)) (justify left))
@@
     )
   )
-  (global_label "LED_POWER" (shape input) (at 156.21 35.56 90) (fields_autoplaced)
-    (effects (font (size 1.27 1.27)) (justify left))
-    (property "Intersheetrefs" "${INTERSHEET_REFS}" (at 156.21 21.7686 90)
-      (effects (font (size 1.27 1.27)) (justify left) hide)
+  (global_label "LED_POWER" (shape input) (at 38.1 143.51 180) (fields_autoplaced)
+    (effects (font (size 1.27 1.27)) (justify right))
+    (property "Intersheetrefs" "${INTERSHEET_REFS}" (at 24.3086 143.51 0)
+      (effects (font (size 1.27 1.27)) (justify right) hide)
     )
   )
@@
     )
   )
-  (global_label "CONN_LED_POWER" (shape output) (at 156.21 40.64 270) (fields_autoplaced)
-    (effects (font (size 1.27 1.27)) (justify right))
-    (property "Intersheetrefs" "${INTERSHEET_REFS}" (at 156.21 60.6605 90)
-      (effects (font (size 1.27 1.27)) (justify right) hide)
+  (global_label "CONN_LED_POWER" (shape output) (at 40.64 143.51 0) (fields_autoplaced)
+    (effects (font (size 1.27 1.27)) (justify left))
+    (property "Intersheetrefs" "${INTERSHEET_REFS}" (at 60.6605 143.51 0)
+      (effects (font (size 1.27 1.27)) (justify left) hide)
     )
   )
@@
     )
   )
-  (symbol (lib_id "Device:LED_Small") (at 161.29 50.8 90) (unit 1)
-    (in_bom yes) (on_board yes) (dnp no) (fields_autoplaced)
-    (property "Reference" "D?" (at 163.83 50.1015 90)
-      (effects (font (size 1.27 1.27)) (justify right))
-    )
-    (property "Value" "LED" (at 163.83 52.6415 90)
-      (effects (font (size 1.27 1.27)) (justify right))
-    )
-    (property "Footprint" "LED_SMD:LED_0603_1608Metric_Pad1.05x0.95mm_HandSolder" (at 161.29 50.8 90)
-      (effects (font (size 1.27 1.27)) hide)
-    )
-    (property "Datasheet" "https://akizukidenshi.com/catalog/g/gI-11882" (at 161.29 50.8 90)
-      (effects (font (size 1.27 1.27)) hide)
-    )
-    (property "LCSC" "" (at 161.29 50.8 0)
-      (effects (font (size 1.27 1.27)) hide)
-    )
-    (pin "1")
-    (pin "2")
-    (instances
-      (project "LaunchController"
-        (path "/628d040b-43bf-4733-804f-091644a90124"
-          (reference "D?") (unit 1)
-        )
-        (path "/628d040b-43bf-4733-804f-091644a90124/e0707eae-5795-481d-8074-cd2b21e2c883"
-          (reference "D18") (unit 1)
-        )
-      )
-    )
-  )
   (symbol (lib_id "power:GND") (at 25.4 55.88 0) (unit 1)
     (in_bom yes) (on_board yes) (dnp no) (fields_autoplaced)
@@
     )
   )
-  (symbol (lib_id "Device:R_Small") (at 161.29 43.18 0) (unit 1)
-    (in_bom yes) (on_board yes) (dnp no) (fields_autoplaced)
-    (property "Reference" "R?" (at 163.83 42.545 0)
-      (effects (font (size 1.27 1.27)) (justify left))
-    )
-    (property "Value" "1kR" (at 163.83 45.085 0)
-      (effects (font (size 1.27 1.27)) (justify left))
-    )
-    (property "Footprint" "Resistor_SMD:R_0603_1608Metric_Pad0.98x0.95mm_HandSolder" (at 161.29 43.18 0)
-      (effects (font (size 1.27 1.27)) hide)
-    )
-    (property "Datasheet" "https://www.chip1stop.com/view/dispDetail/DispDetail?partId=ROHM-0021097" (at 161.29 43.18 0)
-      (effects (font (size 1.27 1.27)) hide)
-    )
-    (property "LCSC" "" (at 161.29 43.18 0)
-      (effects (font (size 1.27 1.27)) hide)
-    )
-    (pin "1")
-    (pin "2")
-    (instances
-      (project "LaunchController"
-        (path "/628d040b-43bf-4733-804f-091644a90124"
-          (reference "R?") (unit 1)
-        )
-        (path "/628d040b-43bf-4733-804f-091644a90124/e0707eae-5795-481d-8074-cd2b21e2c883"
-          (reference "R27") (unit 1)
-        )
-      )
-    )
-  )
   (symbol (lib_id "power:GND") (at 252.73 55.88 0) (unit 1)
     (in_bom yes) (on_board yes) (dnp no) (fields_autoplaced)
@@
         )
       )
-    )
-  )
-  (symbol (lib_id "power:GND") (at 161.29 55.88 0) (unit 1)
-    (in_bom yes) (on_board yes) (dnp no) (fields_autoplaced)
-    (property "Reference" "#PWR?" (at 161.29 62.23 0)
-      (effects (font (size 1.27 1.27)) hide)
-    )
-    (property "Value" "GND" (at 161.29 60.96 0)
-      (effects (font (size 1.27 1.27)))
-    )
-    (property "Footprint" "" (at 161.29 55.88 0)
-      (effects (font (size 1.27 1.27)) hide)
-    )
-    (property "Datasheet" "" (at 161.29 55.88 0)
-      (effects (font (size 1.27 1.27)) hide)
-    )
-    (pin "1")
-    (instances
-      (project "LaunchController"
-        (path "/628d040b-43bf-4733-804f-091644a90124"
-          (reference "#PWR?") (unit 1)
-        )
-        (path "/628d040b-43bf-4733-804f-091644a90124/e0707eae-5795-481d-8074-cd2b21e2c883"
-          (reference "#PWR06") (unit 1)
-        )
-      )

Commit message: 選定部品を調整
Parts:
- D? (x14): value LED -> LED_O
- D? (x4): value LED -> LED_B
- D? (x2): value LED -> LED_R
- D? (x2): value LED -> LED_G
