File: KiCad/LaunchController/Peripheral.kicad_sch (KiCad schematic)
At the start: 8 parts, among them J15 CONN_AUDIO, J16 CONN_SPEAKER, J2 CONN_RS485, U2 24LC256, U6 DFPlayer, U7 LTC485CN8#PBF

Commit message: KiCad9.0に対応
Parts:
- renumbered D1 to D18, J15 to J10, J16 to J12, J2 to J15, R28 to R26, U2 to U7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
