File: KiCad/SatelliteController/Power.kicad_sch (KiCad schematic)
At the start: 39 parts, among them J1 DC_IN, J1 FROM_CONVERTER, J1 TO_CONVERTER, Q1 TJ8S06M3L, Q2 2SC3325-Y, Q3 TJ8S06M3L, U3 INA219BIDCNT, U5 INA219BIDCNT

Commit message: ランコンのKiCadプロジェクトをコピーしてサテコンを作成
Parts:
- removed R11, R16: 12kR, Resistor_SMD:R_0603_1608Metric_Pad0.98x0.95mm_HandSolder, symbol Device:R_Small
- removed R12, R17: 2kR, Resistor_SMD:R_0603_1608Metric_Pad0.98x0.95mm_HandSolder, symbol Device:R_Small
- C15, C17: footprint Capacitor_SMD:C_0603_1608Metric_Pad1.08x0.95mm_HandSolder -> Capacitor_SMD:C_1206_3216Metric_Pad1.33x1.80mm_HandSolder
- R6: value 2.2kR -> 10kR
Connections:
- net +5V: now also R29.2; no longer TH1.1
- net GND: now also TH1.2; no longer R29.1
- net VREF_THERMISTOR: now also R29.1, TH1.1; no longer R29.2, TH1.2
Other:
- note removed: "VOLTAGE MONITOR"
- moved on the sheet: C14, C5, R10, R21, R23, R24, R29, R7, R9, TH1, U3, U5

Commit message: サテコンのクリスマスツリーを削除
Parts:
- renumbered C1 to C12, C5 to C13, C15 to C14, C16 to C15, C17 to C16, C18 to C17, C14 to C18, D6 to D5, D5 to D6, J1 to J4, J1 to J5, J1 to J6, Q3 to Q2, Q2 to Q3, R3 to R11, R4 to R12, R7 to R13, R6 to R14, R9 to R15, R10 to R16, R5 to R17, R21 to R18, R23 to R21, R24 to R22, R29 to R25, TP8 to TP2, TP15 to TP3, TP2 to TP4, U3 to U4

Commit message: 電磁弁制御回路を整理
Parts:
- renumbered C12 to C11, C14 to C12, C15 to C13, C16 to C14, C17 to C15, C13 to C16, C18 to C17, D4 to D5, D5 to D7, J5 to J4, J6 to J5, J4 to J6, Q3 to Q2, Q2 to Q3, R11 to R12, R12 to R13, R17 to R14, R14 to R15, R25 to R16, R13 to R17, R15 to R19, R16 to R20

Commit message: ガーバーを出力
Parts:
- R12: value 5.6R -> 5.6kR
- R13: value 3.3R -> 3.3kR
Changed lines of the file:
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@@
 			)
 		)
-		(property "Value" "5.6R"
+		(property "Value" "5.6kR"
 			(at 82.55 33.655 0)
 			(effects
@@
 			)
 		)
-		(property "Value" "3.3R"
+		(property "Value" "3.3kR"
 			(at 92.71 43.815 0)
 			(effects
