File: KiCad/BranchAdapter/BranchAdapter.kicad_pcb (KiCad board)
At the start: 2 copper layers, 93 x 32 mm, 22 parts, among them J1 Conn_01x02, J10 Conn_01x10, J2 Conn_01x02, J3 Conn_01x02, J5 Conn_01x02, J6 Conn_01x02, J7 Conn_01x02, J9 Conn_01x02

Commit message: ボード図を更新
Routing:
- net SV_PURGE: track 103.1 -> 103.4 mm, vias 0 -> 1
- net +12V: vias 0 -> 95
- added copper zone on B.Cu, net +12V
- added copper zone on F.Cu, net +12V
