File: KiCad/THRValveControlModule/THRValveControlModule.kicad_pcb (KiCad board)
At the start: 2 copper layers, 99 x 75 mm, 54 parts, among them J1 B4B-XH-A(LF)(SN), J2 B3B-XH-A(LF)(SN), J3 B3B-XH-A(LF)(SN), J4 XT30PW-M, J5 DF51A-4P-2DSA, J6 SSD1306, J7 DF51A-8DP-2DS, Q1 IRLML6344TRPBFTR, U1 XIAO-RA4M1-SMD, U10 MB85RQ8MX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

Commit message: Build-1 は失敗
Parts:
- removed END 120R: IS-2235, Button_Switch_THT:SW_CK_JS202011CQN_DPDT_Straight
- removed SW A: SKRPACE010, TSRP_Button_Switch_SMD:SKRPACE010
- added D3: RB160M-30TR, Diode_SMD:D_SOD-123, F.Cu at (49.2, 74.3)
- added D7: RB160M-30TR, Diode_SMD:D_SOD-123, F.Cu at (49.2, 77.6)
- added D8: RB160M-30TR, Diode_SMD:D_SOD-123, F.Cu at (49.2, 81.0)
- added SW1: IS-2235, Button_Switch_THT:SW_CK_JS202011CQN_DPDT_Straight, F.Cu at (61.9, 77.4)
- added SW2: SKRPACE010, TSRP_Button_Switch_SMD:SKRPACE010, F.Cu at (80.6, 50.2)
- added SW4: SW_DPDT_x2, Button_Switch_THT:SW_E-Switch_EG1271_SPDT, F.Cu at (44.4, 91.7)
- added U11: STM32F446RETx, Package_QFP:LQFP-64_10x10mm_P0.5mm, F.Cu at (39.1, 76.5)
- U1: value XIAO-RA4M1-SMD -> CH340K; footprint TSRP_Seeed_XIAO:XIAO-RA4M1-SMD -> Package_SO:SSOP-10-1EP_3.9x4.9mm_P1mm_EP2.1x3.3mm
- U7: value BP5293-50 -> AZ1117CH-3.3TRG1; footprint TSRP_IC:BP5293-50 -> Package_TO_SOT_SMD:SOT-223-3_TabPin2
- moved U6 189.6 mm to (24.7, 29.5), turned to 0 degrees
- moved H1 182.5 mm to (27.9, 73.2)
- moved H2 168.2 mm to (27.9, 81.2)
- moved J4 167.4 mm to (34.1, 64.5), turned to 0 degrees
- moved D5 164.4 mm to (51.4, 29.5), turned to 0 degrees
- moved G*** 163.4 mm to (132.5, -47.6)
- moved G*** 163.4 mm to (162.3, -18.7)
- moved G*** 163.4 mm to (101.0, -84.1)
- moved U7 157.0 mm to (36.8, 87.9)
- moved D1 152.5 mm to (49.2, 70.9)
- moved U1 141.0 mm to (46.3, 86.9), turned to 0 degrees
- moved C9 137.7 mm to (61.3, 44.4), turned to 0 degrees
- moved C8 135.7 mm to (61.3, 41.9), turned to 0 degrees
- moved R1 129.5 mm to (34.0, 93.3), turned to 0 degrees
- moved C7 128.7 mm to (61.3, 39.4), turned to 0 degrees
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Connections:
- D1 pad 1: Net-(D1-K) -> unconnected-(D1-K-Pad1)
- U1 pad 1: RS485_EN -> USB_D+
- U1 pad 10: CAN_RXD -> +3.3V
- U1 pad 11: CAN_TXD -> GND
- U1 pad 2: Umbilical_GseValve -> USB_D-
- U1 pad 3: Umbilical_GseIgnition -> GND
- U1 pad 4: ServoB_PWM -> unconnected-(U1-~{DTR}-Pad4)
- U1 pad 5: I2C_SDA -> unconnected-(U1-~{CTS}-Pad5)
- U1 pad 6: I2C_SCL -> unconnected-(U1-~{RTS}-Pad6)
- U1 pad 7: RS485_DI -> +3.3V
- U1 pad 8: RS485_RO -> UART1_TX
- U1 pad 9: ServoA_PWM -> UART1_RX
- U7 pad 1: SC8721_VOUT -> Net-(D3-K)
- U7 pad 3: +5V -> +3.3V
Routing:
- net +3.3V: track 221.3 -> 0.00 mm, vias 5 -> 0
- net +5V: track 192.0 -> 0.00 mm, vias 2 -> 0
- net RS485_EN: track 136.0 -> 0.00 mm, vias 4 -> 0
- net RS485_DI: track 115.1 -> 0.00 mm, vias 4 -> 0
- net RS485_RO: track 94.1 -> 0.00 mm, vias 2 -> 0
- net ServoB_PWM: track 93.3 -> 0.00 mm, vias 5 -> 0
- net SC8721_VOUT: track 89.2 -> 0.00 mm
- net Periferal_Speaker: track 87.9 -> 0.00 mm, vias 2 -> 0
- net I2C_SCL: track 85.2 -> 0.00 mm, vias 2 -> 0
- net CAN_RXD: track 84.6 -> 0.00 mm, vias 2 -> 0
- net I2C_SDA: track 83.5 -> 0.00 mm, vias 2 -> 0
- net CAN_TXD: track 81.8 -> 0.00 mm, vias 2 -> 0
- net SPI_FeRAM0_~{CS}: track 79.8 -> 0.00 mm, vias 4 -> 0
- net SPI_SCLK: track 79.4 -> 0.00 mm, vias 2 -> 0
- net SPI_SDO: track 70.7 -> 0.00 mm, vias 3 -> 0
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- removed copper zone on B.Cu, net GND
- removed copper zone on F.Cu, net GND
- removed copper zone on F.Cu, net Net-(D5-A)
- removed copper zone on F.Cu, net SC8721_VIN
- removed copper zone on F.Cu, net SC8721_VOUT
