File: KiCad/THRValveControlModule/THRValveControlModule.kicad_sch (KiCad schematic)
At the start: 9 parts, among them U1 XIAO-RA4M1-SMD

Commit message: とりあえずプッシュ
Parts:
- removed U1: XIAO-RA4M1-SMD, TSRP_Seeed_XIAO:XIAO-RA4M1-SMD, symbol TSRP_Seeed_Studio_XIAO_Series:XIAO-RA4M1-SMD
- added C10, C11, C12, C14, C15, C3, C5: 0.1uF, symbol Device:C_Small
- added C13: 4.7uF, symbol Device:C_Small
- added D3: D_Schottky, symbol Device:D_Schottky
- added J8: USB_C_Receptacle_USB2.0_14P, symbol Connector:USB_C_Receptacle_USB2.0_14P
- added R14: 10k, symbol Device:R_Small
- added R16, R17: 5.1k, symbol Device:R_Small
- added U1: CH340K, Package_SO:SSOP-10-1EP_3.9x4.9mm_P1mm_EP2.1x3.3mm, symbol Interface_USB:CH340K
- added U11: STM32F446RETx, Package_QFP:LQFP-64_10x10mm_P0.5mm, symbol MCU_ST_STM32F4:STM32F446RETx
Connections:
- net +3.3V: now also C10.1, C11.1, C12.1, C3.1, C5.1, U1.10 (V3), U1.7 (VCC), U11.1 (VBAT), U11.13 (VDDA), U11.19 (VDD), U11.32 (VDD), U11.48 (VDD), U11.64 (VDD)
- net +5V: now also C15.1, D3.2 (A), J8.A4 (VBUS), J8.A9 (VBUS), J8.B4 (VBUS), J8.B9 (VBUS)
- net GND: now also C10.2, C11.2, C12.2, C13.2, C14.2, C15.2, C3.2, C5.2, J8.A1 (GND), J8.A12 (GND), J8.B1 (GND), J8.B12 (GND), J8.S1 (SHIELD), R16.2, R17.2, U1.11 (GND), U1.3 (GND), U11.12 (VSSA), U11.18 (VSS), U11.31 (VSS), U11.47 (VSS), U11.63 (VSS)
- new net: C13.1, U11.30 (VCAP_1)
- new net: J8.B5 (CC2), R16.1
- new net: J8.A5 (CC1), R17.1
- new net NRST: C14.1, U1.4 (~{DTR})
- new net UART1_RX: U1.9 (RXD)
- new net UART1_TX: U1.8 (TXD)
- new net USB_D+: J8.A6 (D+), J8.B6 (D+), U1.1 (UD+)
- new net USB_D-: J8.A7 (D-), J8.B7 (D-), U1.2 (UD-)
- no-connect marks 7 -> 2
Other:
- note added: "参考資料 | https://github.com/TanoRoboRCJ/Hardware/blob/main/Archive/PCB/01-main.pdf"
- moved on the sheet: D1, H1, H2, H3, H4, R1, R15, R2

Commit message: Build-1 は失敗
Parts:
- removed D3: D_Schottky, symbol Device:D_Schottky
- added C16, C17: 0.1uF, symbol Device:C_Small
- added C19: 4.7uF, symbol Device:C_Small
- added C20: 30pF, symbol Device:C_Small
- added C21: 10uF, symbol Device:C_Small
- added C22: 22uF, symbol Device:C_Small
- added D3, D7, D8: RB160M-30TR, Diode_SMD:D_SOD-123, symbol Device:D_Schottky_Small
- added D4: Blue, symbol Device:LED_Small
- added D9: green, symbol Device:LED_Small
- added FB1: 120, symbol Device:FerriteBead_Small
- added J9: ST-LINK, symbol Connector_Generic:Conn_02x07_Odd_Even
- added JP2: SB, Jumper:SolderJumper-2_P1.3mm_Bridged_RoundedPad1.0x1.5mm, symbol Jumper:SolderJumper_2_Bridged
- added R18: 0, symbol Device:R_Small
- added R19, R20, R21, R22: 10k, symbol Device:R_Small
- added SW3: SW_MEC_5E, symbol Switch:SW_MEC_5E
- added SW4: SW_DPDT_x2, Button_Switch_THT:SW_E-Switch_EG1271_SPDT, symbol Switch:SW_DPDT_x2
- added U7: AZ1117CH-3.3TRG1, Package_TO_SOT_SMD:SOT-223-3_TabPin2, symbol Regulator_Linear:AZ1117CH2-3.3
- added Y1: 8MHz, symbol Device:Crystal_Small
- C14: value 0.1uF -> 1uF
- C3: value 0.1uF -> 30pF
Connections:
- net +3.3V: now also C14.1, C15.1, C17.1, C19.1, C22.1, D3.2 (A), FB1.1, J9.3 (Pin_3), JP2.1 (A), R20.2, SW4.1 (A), U7.3 (OUT); no longer C3.1
- net +5V: now also D7.2 (A), R22.1; no longer C15.1
- net GND: now also C16.2, C17.2, C19.2, C20.2, C21.2, C22.2, D4.1 (K), D9.1 (K), J9.11 (Pin_11), J9.5 (Pin_5), J9.7 (Pin_7), R19.2, SW3.1, SW3.2, U7.2 (GND)
- net NRST: now also U11.7 (NRST), C16.1, R20.1, SW3.3 (K), SW3.4 (A); no longer C14.1, U1.4 (~{DTR})
- net USART2_TX_16: now reaches U11.16 (PA2)
- net USART2_TX_16: now also J9.14 (Pin_14)
- net USART2_RX_17: now reaches U11.17 (PA3)
- net USART2_RX_17: now also J9.13 (Pin_13)
- net at U11.21 (PA5): now also R21.1
- net SWDIO_46: now reaches U11.46 (PA13)
- net SWDIO_46: now also J9.4 (Pin_4)
- net SWCLK_49: now reaches U11.49 (PA14)
- net SWCLK_49: now also J9.6 (Pin_6)
- net at U11.5 (PH0): now also C20.1, Y1.1
- net SWO_55: now reaches U11.55 (PB3)
- net SWO_55: now also J9.8 (Pin_8)
- net at U11.6 (PH1): now also R18.2
- net BOOT0: now reaches U11.60 (BOOT0)
- net BOOT0: now also R19.1, SW4.2 (B)
- new net: FB1.2, JP2.2 (B)
- new net: C21.1, D3.1 (K), D7.1 (K), D8.1 (K), U7.1 (IN)
- new net: C3.1, R18.1, Y1.2
- new net: D9.2 (A), R22.2
- new net: D4.2 (A), R21.2
- new net NRST_7: J9.12 (Pin_12)
- new net SC8721_VOUT: D8.2 (A)
- no-connect marks 2 -> 8
Other:
- note added: "12Vくらい"
- note added: "C13 マイコン近くに"
- note added: "C16 マイコン近くに"
- note added: "STDC14 に従って作成 書き込み用"
- note added: "クロス接続"
- note added: "参考資料 | STM32で最小構成のマイコンボードを作る（UART書き込み）"
- note added: "参考資料 | STM32を動かすための最低限の回路"
- note added: "参考資料 | STM32マイコンを用いて自作基板をつくろう"
- note added: "外部水晶発振子はマイコン近くに"
- note added: "最短でVSSA(12)へと接続"
- moved on the sheet: C10, C11, C12, C13, C5, H1, H2, H3, H4, J8, R16, R17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
