File: KiCad/THRValveControlModule/powerManagement.kicad_sch (KiCad schematic)
At the start: 5 parts, among them J4 XT30PW-M, U6 SC8721, U7 BP5293-50

Commit message: Build-1 は失敗
Parts:
- removed U7: BP5293-50, TSRP_IC:BP5293-50, symbol TSRP_IC:BP5293-50
