File: KiCad/LaunchController2.0/Extension.kicad_sch (KiCad schematic)
At the start: 4 parts, among them J10 CONN_PANEL_BAORD_2, J7 CONN_STATUS_PANEL, J8 CONN_BOARD_3, J9 CONN_PANEL_BAORD_1

Commit message: Build-1いったん完成
Parts:
- J10: value CONN_PANEL_BAORD_2 -> CONN_PANEL_BOARD_2
- J9: value CONN_PANEL_BAORD_1 -> CONN_PANEL_BOARD_1
Changed lines of the file:
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@@
 		(fields_autoplaced yes)
 		(property "Reference" "J10"
-			(at 133.35 25.4 0)
+			(at 133.35 24.13 0)
 			(effects
 				(font
@@
 			)
 		)
-		(property "Value" "CONN_PANEL_BAORD_2"
-			(at 133.35 27.94 0)
+		(property "Value" "CONN_PANEL_BOARD_2"
+			(at 133.35 26.67 0)
 			(effects
 				(font
@@
 		(fields_autoplaced yes)
 		(property "Reference" "J9"
-			(at 91.44 31.75 0)
+			(at 91.44 30.48 0)
 			(effects
 				(font
@@
 			)
 		)
-		(property "Value" "CONN_PANEL_BAORD_1"
-			(at 91.44 34.29 0)
+		(property "Value" "CONN_PANEL_BOARD_1"
+			(at 91.44 33.02 0)
 			(effects
 				(font
