File: KiCad/LaunchController2.0/Extension.kicad_sch (KiCad schematic)
At the start: 4 parts, among them J10 CONN_PANEL_BOARD_2, J7 CONN_STATUS_PANEL, J8 CONN_BOARD_3, J9 CONN_PANEL_BOARD_1

Commit message: シルクなどを調整
Parts:
- J10: Digikey_PN (none) -> 26-DF51A-22DP-2DS(20)-ND
- J7: Mouser_PN (none) -> 798-DF51A14DP2DS50
- J8: Mouser_PN (none) -> 798-DF51A-6DP-2DSA
- J9: Digikey_PN (none) -> 26-DF51A-18DP-2DS(20)-ND
Other:
- company: (none) -> Tokai Student Rocket Project
- title: (none) -> Gen6 GSE Launch Controller 2.0

Commit message: とりあえずプッシュ
Parts:
- J10: DigiKey_PN (none) -> 26-DF51A-22DP-2DS(20)-ND
- J9: DigiKey_PN (none) -> 26-DF51A-18DP-2DS(20)-ND
Changed lines of the file:
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@@
+			)
+		)
+		(property "DigiKey_PN" "26-DF51A-22DP-2DS(20)-ND"
+			(at 133.35 58.42 0)
+			(effects
+				(font
+					(size 1.27 1.27)
+				)
+				(hide yes)
 			)
 		)
@@
 			(at 91.44 59.69 0)
 			(effects
+				(font
+					(size 1.27 1.27)
+				)
+				(hide yes)
+			)
+		)
+		(property "DigiKey_PN" "26-DF51A-18DP-2DS(20)-ND"
+			(at 91.44 59.69 0)
+			(effects
