File: KiCad/LaunchController2.0/Indicator.kicad_sch (KiCad schematic)
At the start: 40 parts

Commit message: シルクなどを調整
Parts:
- added D26: LED_O, LED_SMD:LED_0603_1608Metric_Pad1.05x0.95mm_HandSolder, symbol Device:LED_Small
- added R66: 1kR, Resistor_SMD:R_0603_1608Metric_Pad0.98x0.95mm_HandSolder, symbol Device:R_Small
- D10, D15, D16, D17, D18, D19, D20, D21, D22, D23, D24, D25, D7, D9: Digikey_PN (none) -> SML-D12D8WT86CCT-ND
- D11, D13: Digikey_PN (none) -> SML-D12U8WT86CCT-ND
- D12, D14: Digikey_PN (none) -> SML-D12P8WT86CCT-ND
- D6: value LED_B -> LED_G; Digikey_PN (none) -> SMLD12BN1WT86CT-ND
- D8: Digikey_PN (none) -> SMLD12BN1WT86CT-ND
- R46: renamed from R45; Digikey_PN (none) -> 2019-RK73H1JTTD1001FCT-ND
- R47: renamed from R46; Digikey_PN (none) -> 2019-RK73H1JTTD5101FCT-ND
- R48: renamed from R47; Digikey_PN (none) -> 2019-RK73H1JTTD1001FCT-ND
- R49: renamed from R48; Digikey_PN (none) -> 2019-RK73H1JTTD5101FCT-ND
- R50: renamed from R49; Digikey_PN (none) -> 2019-RK73H1JTTD1001FCT-ND
- R51: renamed from R50; Digikey_PN (none) -> 2019-RK73H1JTTD1001FCT-ND
- R52: renamed from R51; Digikey_PN (none) -> 2019-RK73H1JTTD1001FCT-ND
- R53: renamed from R52; Digikey_PN (none) -> 2019-RK73H1JTTD1001FCT-ND
- R54: renamed from R53; Digikey_PN (none) -> 2019-RK73H1JTTD1001FCT-ND
- R55: renamed from R54; Digikey_PN (none) -> 2019-RK73H1JTTD1001FCT-ND
- R56: renamed from R55; Digikey_PN (none) -> 2019-RK73H1JTTD1001FCT-ND
- R57: renamed from R56; Digikey_PN (none) -> 2019-RK73H1JTTD1001FCT-ND
- R58: renamed from R57; Digikey_PN (none) -> 2019-RK73H1JTTD1001FCT-ND
- R59: renamed from R58; Digikey_PN (none) -> 2019-RK73H1JTTD1001FCT-ND
- R60: renamed from R59; Digikey_PN (none) -> 2019-RK73H1JTTD1001FCT-ND
- R61: renamed from R60; Digikey_PN (none) -> 2019-RK73H1JTTD1001FCT-ND
- R62: renamed from R61; Digikey_PN (none) -> 2019-RK73H1JTTD1001FCT-ND
- R63: renamed from R62; Digikey_PN (none) -> 2019-RK73H1JTTD1001FCT-ND
- R64: renamed from R63; Digikey_PN (none) -> 2019-RK73H1JTTD1001FCT-ND
- R65: renamed from R64; Digikey_PN (none) -> 2019-RK73H1JTTD1001FCT-ND
Connections:
- net +5V: now also D26.2 (A)
- new net: D26.1 (K), R66.1
- new net LED_USB_TXLED: R66.2
Other:
- company: (none) -> Tokai Student Rocket Project
- title: (none) -> Gen6 GSE Launch Controller 2.0
- moved on the sheet: D11, D13, D8, R48, R51, R53

Commit message: BOM作成
Parts:
- D11: renamed from D10; Digikey_PN SML-D12D8WT86CCT-ND -> SML-D15DWT86CCT-ND
- D16: renamed from D15; Digikey_PN SML-D12D8WT86CCT-ND -> SML-D15DWT86CCT-ND
- D17: renamed from D16; Digikey_PN SML-D12D8WT86CCT-ND -> SML-D15DWT86CCT-ND
- D18: renamed from D17; Digikey_PN SML-D12D8WT86CCT-ND -> SML-D15DWT86CCT-ND
- D19: renamed from D18; Digikey_PN SML-D12D8WT86CCT-ND -> SML-D15DWT86CCT-ND
- D20: renamed from D19; Digikey_PN SML-D12D8WT86CCT-ND -> SML-D15DWT86CCT-ND
- D21: renamed from D20; Digikey_PN SML-D12D8WT86CCT-ND -> SML-D15DWT86CCT-ND
- D22: renamed from D21; Digikey_PN SML-D12D8WT86CCT-ND -> SML-D15DWT86CCT-ND
- D23: renamed from D22; Digikey_PN SML-D12D8WT86CCT-ND -> SML-D15DWT86CCT-ND
- D24: renamed from D23; Digikey_PN SML-D12D8WT86CCT-ND -> SML-D15DWT86CCT-ND
- D25: renamed from D24; Digikey_PN SML-D12D8WT86CCT-ND -> SML-D15DWT86CCT-ND
- D26: renamed from D25; Digikey_PN SML-D12D8WT86CCT-ND -> SML-D15DWT86CCT-ND
- D6: Digikey_PN SMLD12BN1WT86CT-ND -> SML-D12P8WT86CCT-ND
- D7, D9: Digikey_PN SML-D12D8WT86CCT-ND -> SML-D15DWT86CCT-ND
- D8: renamed from D26; Digikey_PN SMLD12BN1WT86CT-ND -> SML-D15DWT86CCT-ND
- renumbered D8 to D10, D11 to D12, D12 to D13, D13 to D14, D14 to D15, R66 to R48, R48 to R50, R50 to R51, R51 to R52, R52 to R53, R53 to R54, R54 to R55, R55 to R56, R56 to R57, R57 to R58, R58 to R59, R59 to R60, R60 to R61, R61 to R62, R62 to R63, R63 to R64, R64 to R65, R65 to R66

Commit message: とりあえずプッシュ
Parts:
- D10: Akiduki_PN (none) -> 103982
- D11, D16, D17, D18, D19, D20, D21, D22, D23, D24, D25, D26, D7, D8, D9: DigiKey_PN (none) -> 160-1434-1-ND
- D12, D14: Akiduki_PN (none) -> 111879
- D13, D15, D6: Akiduki_PN (none) -> 111878
- R46, R48, R50, R51, R52, R53, R54, R55, R56, R57, R58, R59, R60, R61, R62, R63, R64, R65, R66: DigiKey_PN (none) -> 2019-RK73H1JTTD1001FCT-ND
- R47, R49: DigiKey_PN (none) -> 2019-RK73H1JTTD5101FCT-ND
