File: KiCad/LaunchController2.0/Peripheral.kicad_sch (KiCad schematic)
At the start: 20 parts, among them J11 CONN_AUDIO, J12 CONN_SPEAKER, J13 CONN_RS485, U10 ADM2582E, U11 24LC256, U8 MB85RQ8MX, U9 DFPlayer

Commit message: シルクなどを調整
Parts:
- added C31, C32: 470pF, Capacitor_SMD:C_1206_3216Metric_Pad1.33x1.80mm_HandSolder, symbol Device:C_Small
- added J13: Conn_01x08, symbol Connector_Generic:Conn_01x08
- added R44: TestPoint_A, Resistor_SMD:R_0805_2012Metric, symbol Device:R_Small
- added R45: TestPoint_B, Resistor_SMD:R_0805_2012Metric, symbol Device:R_Small
- C26, C27: value 0.1uF -> 10uF; footprint Capacitor_SMD:C_0603_1608Metric_Pad1.08x0.95mm_HandSolder -> Capacitor_SMD:C_0805_2012Metric_Pad1.18x1.45mm_HandSolder; Digikey_PN (none) -> 490-GCM21BC71C106KE36KCT-ND
- C29, C30: value 0.01uF -> 0.1uF; Digikey_PN (none) -> 490-4781-1-ND
- C33: renamed from C31; Digikey_PN (none) -> 490-8020-1-ND
- C34: renamed from C32; value 0.01uF -> 10uF; footprint Capacitor_SMD:C_0603_1608Metric_Pad1.08x0.95mm_HandSolder -> Capacitor_SMD:C_0805_2012Metric_Pad1.18x1.45mm_HandSolder; Digikey_PN (none) -> 490-4781-1-ND
- C35: renamed from C34; value 0.01uF -> 10uF; footprint Capacitor_SMD:C_0603_1608Metric_Pad1.08x0.95mm_HandSolder -> Capacitor_SMD:C_0805_2012Metric_Pad1.18x1.45mm_HandSolder; Digikey_PN (none) -> 490-4781-1-ND
- C36: renamed from C33; Digikey_PN (none) -> 490-8020-1-ND
- D5: Akiduki_PN (none) -> 106014
- FB1, FB2: Digikey_PN (none) -> 445-MMZ1608S202ATA00CT-ND
- J11, J12: Digikey_PN (none) -> 2946-2601-3102-ND
- J14: renamed from J13; Digikey_PN (none) -> 2946-2601-3104-ND
- R43: renamed from R44; Digikey_PN (none) -> 13-RC0603FR-13120RLCT-ND
- U10: value ADM2582E -> ADM2587EBRWZ; Akiduki_PN (none) -> 113300
- U11: Akiduki_PN (none) -> 100705
- U9: Akiduki_PN (none) -> 112544
Connections:
- net GND: now also C31.1
- net GND2: now also C32.2
- net Visoin: now also C35.2; no longer C36.2
- net Visoout: now also C36.2; no longer C35.2
- net at R43.1, U10.15 (Z), U10.17 (B): now also R45.1; no longer J14.3 (Pin_3)
- net at R43.2, U10.13 (Y), U10.18 (A): now also R44.2; no longer J14.2 (Pin_2)
- new net: C31.2, C32.1
- new net: J14.2 (Pin_2), R44.1
- new net: J14.3 (Pin_3), R45.2
Other:
- note added: "丸ピンICソケット（BOM用）"
- company: (none) -> Tokai Student Rocket Project
- title: (none) -> Gen6 GSE Launch Controller 2.0
- moved on the sheet: C35, C36, J14

Commit message: BOM作成
Parts:
- removed C28: 0.1uF, Capacitor_SMD:C_0603_1608Metric_Pad1.08x0.95mm_HandSolder, symbol Device:C_Small
- removed U8: MB85RQ8MX, Package_SO:SOIC-16W_7.5x10.3mm_P1.27mm, symbol TSRP_IC:MB85RQ8MX
- C26, C27: Akiduki_PN (none) -> 113388; Digikey_PN 490-GCM21BC71C106KE36KCT-ND -> (none)
- C28: renamed from C29; Akiduki_PN (none) -> 114559; Digikey_PN 490-4781-1-ND -> (none)
- C29: renamed from C30; Akiduki_PN (none) -> 114559; Digikey_PN 490-4781-1-ND -> (none)
- C32: renamed from C33; Akiduki_PN (none) -> 114559; Digikey_PN 490-8020-1-ND -> (none)
- C33: renamed from C34; Akiduki_PN (none) -> 113388; Digikey_PN 490-4781-1-ND -> (none)
- C34: renamed from C35; Akiduki_PN (none) -> 113388; Digikey_PN 490-4781-1-ND -> (none)
- C35: renamed from C36; Akiduki_PN (none) -> 114559; Digikey_PN 490-8020-1-ND -> (none)
- R43: footprint Resistor_SMD:R_0603_1608Metric_Pad0.98x0.95mm_HandSolder -> Resistor_SMD:R_0805_2012Metric_Pad1.20x1.40mm_HandSolder; Digikey_PN 13-RC0603FR-13120RLCT-ND -> 2019-RK73H2ATTD1200FCT-ND
- renumbered C31 to C30, C32 to C31, U11 to U10, U9 to U8, U10 to U9
Other:
- note removed: "FeRAM0"

Commit message: とりあえずプッシュ
Parts:
- C30, C31: DigiKey_PN (none) -> 445-5785-1-ND
- FB1, FB2: DigiKey_PN (none) -> 445-MMZ1608S202ATA00CT-ND
- J11, J12: DigiKey_PN (none) -> 2946-2601-3102-ND
- J14: DigiKey_PN (none) -> 2946-2601-3104-ND
- R43: DigiKey_PN (none) -> 2019-RK73H2ATTD1200FCT-ND
Changed lines of the file:
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@@
 			)
 		)
+		(property "DigiKey_PN" "445-5785-1-ND"
+			(at 101.6 132.08 90)
+			(effects
+				(font
+					(size 1.27 1.27)
+				)
+				(hide yes)
+			)
+		)
 		(pin "1"
 		)
@@
 			)
 		)
+		(property "DigiKey_PN" "2019-RK73H2ATTD1200FCT-ND"
+			(at 132.08 104.14 0)
+			(effects
+				(font
+					(size 1.27 1.27)
+				)
+				(hide yes)
+			)
+		)
 		(pin "1"
 		)
@@
 			)
 		)
+		(property "DigiKey_PN" "2946-2601-3102-ND"
+			(at 24.13 53.34 0)
+			(effects
+				(font
+					(size 1.27 1.27)
+				)
+				(hide yes)
+			)
+		)
 		(pin "1"
 		)
@@
 			)
 		)
+		(property "DigiKey_PN" "2946-2601-3104-ND"
+			(at 166.37 102.87 0)
+			(effects
+				(font
+					(size 1.27 1.27)
+				)
+				(hide yes)
+			)
+		)
 		(pin "1"
 		)
@@
 			)
 		)
+		(property "DigiKey_PN" "445-MMZ1608S202ATA00CT-ND"
+			(at 173.99 119.38 90)
+			(effects
+				(font
+					(size 1.27 1.27)
+				)
+				(hide yes)
+			)
+		)
 		(pin "1"
 		)
@@
 			)
 		)
+		(property "DigiKey_PN" "445-5785-1-ND"
+			(at 111.76 132.08 90)
+			(effects
+				(font
+					(size 1.27 1.27)
+				)
+				(hide yes)
+			)
+		)
 		(pin "1"
 		)
@@
 			)
 		)
+		(property "DigiKey_PN" "445-MMZ1608S202ATA00CT-ND"
+			(at 173.99 127 90)
+			(effects
+				(font
+					(size 1.27 1.27)
+				)
+				(hide yes)
+			)
+		)
 		(pin "1"
 		)
@@
 			(at 24.13 35.56 0)
 			(effects
+				(font
+					(size 1.27 1.27)
+				)
+				(hide yes)
+			)
+		)
+		(property "DigiKey_PN" "2946-2601-3102-ND"
+			(at 24.13 35.56 0)
+			(effects
