File: KiCad/LaunchController2.0/Power.kicad_sch (KiCad schematic)
At the start: 45 parts, among them J4 TO_CONVERTER, J5 FROM_CONVERTER, J6 DC_IN, Q1 TJ8S06M3L, Q2 2SC3325-Y, Q3 TJ8S06M3L, U4 TPS2116DRL, U5 NJM7805SDL1, U6 INA219BIDCNT, U7 INA219BIDCNT

Commit message: シルクなどを調整
Parts:
- removed D3: GS1010FL, Diode_SMD:D_SOD-123F, symbol Device:D_Small
- added D3: SS2040FL, TSRP_Diode:SOD-123FL_Handsolder, symbol Device:D_Schottky_Small
- C12, C16, C19, C23, C25: Digikey_PN (none) -> 490-8020-1-ND
- C13, C14: Digikey_PN (none) -> 490-GCM188D71H105KE36JCT-ND
- C15, C17: Akiduki_PN (none) -> 117338
- C18, C22, C24: Digikey_PN (none) -> 490-GCM21BC71C106KE36KCT-ND
- C20, C21: value uF -> 0.1uF; Digikey_PN (none) -> 490-8020-1-ND
- D4: Digikey_PN (none) -> SML-D12Y8WT86CCT-ND
- J4, J5, J6: Digikey_PN (none) -> 2946-2601-3102-ND
- Q1, Q3: Akiduki_PN (none) -> 113964
- Q2: Akiduki_PN (none) -> 100628
- R29: renamed from R30; Digikey_PN (none) -> 2019-RK73H1JTTD1002FCT-ND
- R30: renamed from R31; Digikey_PN (none) -> 2019-RK73H1JTTD5601FCT-ND
- R31: renamed from R32; Digikey_PN (none) -> 2019-RK73H1JTTD3301FCT-ND
- R32: renamed from R33; Digikey_PN (none) -> 2019-RK73H1JTTD1002FCT-ND
- R33: renamed from R34; Digikey_PN (none) -> 2019-RK73H1JTTD1002FCT-ND
- R34: renamed from R35; Digikey_PN (none) -> 2019-RK73H1JTTD3483FCT-ND
- R35: renamed from R36; Digikey_PN (none) -> 2019-RK73H1JTTD1003FCT-ND
- R36: renamed from R37; value 100 -> 100R; Digikey_PN (none) -> 2019-RK73H1JTTD1000FCT-ND
- R37: renamed from R38; value 0R -> 10R; Digikey_PN (none) -> 2019-RK73H1JTTD10R0FCT-ND
- R38: renamed from R39; footprint Resistor_SMD:R_2816_7142Metric_Pad3.20x4.45mm_HandSolder -> Resistor_SMD:R_2512_6332Metric_Pad1.40x3.35mm_HandSolder; Digikey_PN (none) -> CRM2512-FX-R100ELFCT-ND
- R39: renamed from R40; value 0R -> 10R; Digikey_PN (none) -> 2019-RK73H1JTTD10R0FCT-ND
- R40: renamed from R41; value 0R -> 10R; Digikey_PN (none) -> 2019-RK73H1JTTD10R0FCT-ND
- R41: renamed from R42; footprint Resistor_SMD:R_2816_7142Metric_Pad3.20x4.45mm_HandSolder -> Resistor_SMD:R_2512_6332Metric_Pad1.40x3.35mm_HandSolder; Digikey_PN (none) -> CRM2512-FX-R100ELFCT-ND
- R42: renamed from R43; value 0R -> 10R; Digikey_PN (none) -> 2019-RK73H1JTTD10R0FCT-ND
- TH1: Digikey_PN (none) -> 2019-RK73H1JTTD1002FCT-ND
- TP1: footprint TestPoint:TestPoint_THTPad_D1.0mm_Drill0.5mm -> TestPoint:TestPoint_Keystone_5005-5009_Compact; Akiduki_PN (none) -> 116480
- TP2, TP3: footprint TestPoint:TestPoint_THTPad_D1.0mm_Drill0.5mm -> TestPoint:TestPoint_Keystone_5005-5009_Compact; Akiduki_PN (none) -> 116434
- TP4: footprint TestPoint:TestPoint_THTPad_D1.0mm_Drill0.5mm -> TestPoint:TestPoint_Keystone_5005-5009_Compact; Akiduki_PN (none) -> 116435
- U4: Digikey_PN (none) -> 296-TPS2116DRLRCT-ND
- U5: Akiduki_PN (none) -> 111237
- U6, U7: Digikey_PN (none) -> 296-27898-1-ND
Connections:
- net +12V: now also D3.1 (K)
- net VIN_5V: now also D3.2 (A)
Other:
- note added: "MULTIPLEXER"
- company: (none) -> Tokai Student Rocket Project
- title: (none) -> Gen6 GSE Launch Controller 2.0

Commit message: BOM作成
Parts:
- C12, C16, C19, C20, C21, C23, C25: Akiduki_PN (none) -> 114559; Digikey_PN 490-8020-1-ND -> (none)
- C13, C14: Akiduki_PN (none) -> 130397; Digikey_PN 490-GCM188D71H105KE36JCT-ND -> (none)
- C18, C22, C24: Akiduki_PN (none) -> 113388; Digikey_PN 490-GCM21BC71C106KE36KCT-ND -> (none)
- D4: value LED_Y -> LED_O; Digikey_PN SML-D12Y8WT86CCT-ND -> SML-D15DWT86CCT-ND
Changed lines of the file:
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@@
 			)
 		)
-		(property "Datasheet" "https://www.digikey.jp/short/ttd7bqv9"
+		(property "Datasheet" "https://akizukidenshi.com/catalog/g/g114559/"
 			(at 233.68 107.95 0)
 			(effects
@@
 			)
 		)
-		(property "Digikey_PN" "490-8020-1-ND"
+		(property "Digikey_PN" ""
+			(at 233.68 107.95 90)
+			(effects
+				(font
+					(size 1.27 1.27)
+				)
+				(hide yes)
+			)
+		)
+		(property "Akiduki_PN" "114559"
 			(at 233.68 107.95 90)
 			(effects
@@
 			)
 		)
-		(property "Datasheet" "https://www.digikey.jp/short/ftvh328f"
+		(property "Datasheet" "https://akizukidenshi.com/catalog/g/g114559/"
 			(at 71.12 33.02 0)
 			(effects
@@
 			)
 		)
-		(property "Digikey_PN" "490-8020-1-ND"
+		(property "Digikey_PN" ""
+			(at 71.12 33.02 0)
+			(effects
+				(font
+					(size 1.27 1.27)
+				)
+				(hide yes)
+			)
+		)
+		(property "Akiduki_PN" "114559"
 			(at 71.12 33.02 0)
 			(effects
@@
 			)
 		)
-		(property "Datasheet" "https://www.digikey.jp/short/fbbb4909"
+		(property "Datasheet" "https://akizukidenshi.com/catalog/g/g113388/"
 			(at 269.24 91.44 0)
 			(effects
@@
 			)
 		)
-		(property "Digikey_PN" "490-GCM21BC71C106KE36KCT-ND"
+		(property "Digikey_PN" ""
+			(at 269.24 91.44 90)
+			(effects
+				(font
+					(size 1.27 1.27)
+				)
+				(hide yes)
+			)
+		)
+		(property "Akiduki_PN" "113388"
 			(at 269.24 91.44 90)
 			(effects
@@
 			)
 		)
-		(property "Datasheet" "https://www.digikey.jp/short/ftvh328f"
+		(property "Datasheet" "https://akizukidenshi.com/catalog/g/g114559/"
 			(at 176.53 40.64 0)
 			(effects
@@
 			)
 		)
-		(property "Digikey_PN" "490-8020-1-ND"
+		(property "Digikey_PN" ""
+			(at 176.53 40.64 0)
+			(effects
+				(font
+					(size 1.27 1.27)
+				)
+				(hide yes)
+			)
+		)
+		(property "Akiduki_PN" "114559"
 			(at 176.53 40.64 0)
 			(effects
@@
 			)
 		)
-		(property "Value" "LED_Y"
+		(property "Value" "LED_O"
 			(at 161.29 105.3464 90)
 			(effects
@@
 			)
 		)
-		(property "Datasheet" "https://www.digikey.jp/short/4nhvjzth"
+		(property "Datasheet" "https://www.digikey.jp/short/3ww5zf50"
 			(at 158.75 104.14 90)
 			(effects
@@
 			)
 		)
-		(property "Digikey_PN" "SML-D12Y8WT86CCT-ND"
+		(property "Digikey_PN" "SML-D15DWT86CCT-ND"
 			(at 158.75 104.14 90)
 			(effects
@@
 			)
 		)
-		(property "Datasheet" "https://www.digikey.jp/short/fbbb4909"
+		(property "Datasheet" "https://akizukidenshi.com/catalog/g/g113388/"
 			(at 254 26.67 0)
 			(effects
@@
 			)
 		)
-		(property "Digikey_PN" "490-GCM21BC71C106KE36KCT-ND"
+		(property "Digikey_PN" ""
+			(at 254 26.67 90)
+			(effects
+				(font
+					(size 1.27 1.27)
+				)
+				(hide yes)
+			)
+		)
+		(property "Akiduki_PN" "113388"
 			(at 254 26.67 90)
 			(effects
@@
 			)
 		)
-		(property "Datasheet" "https://www.digikey.jp/short/2jznv97v"
+		(property "Datasheet" "https://akizukidenshi.com/catalog/g/g130397/"
 			(at 91.44 102.87 0)
 			(effects
@@
 			)
 		)
-		(property "Digikey_PN" "490-GCM188D71H105KE36JCT-ND"
+		(property "Digikey_PN" ""
+			(at 91.44 102.87 0)
+			(effects
+				(font
+					(size 1.27 1.27)
+				)
+				(hide yes)
+			)
+		)
+		(property "Akiduki_PN" "130397"
 			(at 91.44 102.87 0)
 			(effects
@@
 			)
 		)
-		(property "Datasheet" "https://www.digikey.jp/short/ttd7bqv9"
+		(property "Datasheet" "https://akizukidenshi.com/catalog/g/g114559/"
 			(at 218.44 43.18 0)
 			(effects
@@
 			)
 		)
-		(property "Digikey_PN" "490-8020-1-ND"
+		(property "Digikey_PN" ""
+			(at 218.44 43.18 90)
+			(effects
+				(font
+					(size 1.27 1.27)
+				)
+				(hide yes)
+			)
+		)
+		(property "Akiduki_PN" "114559"
 			(at 218.44 43.18 90)
 			(effects
@@
 			)
 		)
-		(property "Datasheet" "https://www.digikey.jp/short/ftvh328f"
+		(property "Datasheet" "https://akizukidenshi.com/catalog/g/g114559/"
 			(at 254 36.83 0)
 			(effects
@@
 			)
 		)
-		(property "Digikey_PN" "490-8020-1-ND"
+		(property "Digikey_PN" ""
+			(at 254 36.83 90)
+			(effects
+				(font
+					(size 1.27 1.27)
+				)
+				(hide yes)
+			)
+		)
+		(property "Akiduki_PN" "114559"
 			(at 254 36.83 90)
 			(effects
@@
 			)
 		)
-		(property "Datasheet" "https://www.digikey.jp/short/ftvh328f"
+		(property "Datasheet" "https://akizukidenshi.com/catalog/g/g114559/"
 			(at 140.97 40.64 0)
 			(effects
@@
 			)
 		)
-		(property "Digikey_PN" "490-8020-1-ND"
+		(property "Digikey_PN" ""
+			(at 140.97 40.64 0)
+			(effects
+				(font
+					(size 1.27 1.27)
+				)
+				(hide yes)
+			)
+		)
+		(property "Akiduki_PN" "114559"
 			(at 140.97 40.64 0)
 			(effects
@@
 			)
 		)
-		(property "Datasheet" "https://www.digikey.jp/short/ftvh328f"
+		(property "Datasheet" "https://akizukidenshi.com/catalog/g/g114559/"
 			(at 269.24 101.6 0)
 			(effects
@@
 			)
 		)
-		(property "Digikey_PN" "490-8020-1-ND"
+		(property "Digikey_PN" ""
+			(at 269.24 101.6 90)
+			(effects
+				(font
+					(size 1.27 1.27)
+				)
+				(hide yes)
+			)
+		)
+		(property "Akiduki_PN" "114559"
 			(at 269.24 101.6 90)
 			(effects
@@
 			)
 		)
-		(property "Datasheet" "https://www.digikey.jp/short/fbbb4909"
+		(property "Datasheet" "https://akizukidenshi.com/catalog/g/g113388/"
 			(at 170.18 102.87 0)
 			(effects
@@
 			)
 		)
-		(property "Digikey_PN" "490-GCM21BC71C106KE36KCT-ND"
+		(property "Digikey_PN" ""
+			(at 170.18 102.87 0)
+			(effects
+				(font
+					(size 1.27 1.27)
+				)
+				(hide yes)
+			)
+		)
+		(property "Akiduki_PN" "113388"
 			(at 170.18 102.87 0)
 			(effects
@@
 			)
 		)
-		(property "Datasheet" "https://www.digikey.jp/short/2jznv97v"
+		(property "Datasheet" "https://akizukidenshi.com/catalog/g/g130397/"
 			(at 127 113.03 0)
 			(effects
@@
 			)
 		)
-		(property "Digikey_PN" "490-GCM188D71H105KE36JCT-ND"
+		(property "Digikey_PN" ""
+			(at 127 113.03 0)
+			(effects
+				(font
+					(size 1.27 1.27)
+				)
+				(hide yes)
+			)
+		)
+		(property "Akiduki_PN" "130397"
 			(at 127 113.03 0)
 			(effects

Commit message: とりあえずプッシュ
Parts:
- D4: DigiKey_PN (none) -> 160-1434-1-ND
- J4, J5, J6: DigiKey_PN (none) -> 2946-2601-3102-ND
- R29, R32, R33, TH1: DigiKey_PN (none) -> 2019-RK73H1JTTD1002FCT-ND
- R30: DigiKey_PN (none) -> 2019-RK73H1JTTD5601FCT-ND
- R31: DigiKey_PN (none) -> 2019-RK73H1JTTD3301FCT-ND
- R34: DigiKey_PN (none) -> 2019-RK73H1JTTD3483FCT-ND
- R35: DigiKey_PN (none) -> 2019-RK73H1JTTD1003FCT-ND
- R36: DigiKey_PN (none) -> 2019-RK73H1JTTD1000FCT-ND
- R37, R39, R40, R42: DigiKey_PN (none) -> 2019-RK73H1JTTD10R0FCT-ND
- R38, R41: Akiduki_PN (none) -> 111878
- U4: DigiKey_PN (none) -> 296-TPS2116DRLRCT-ND
- U6, U7: DigiKey_PN (none) -> 296-27898-1-ND
Changed lines of the file:
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@@
 			)
 		)
+		(property "DigiKey_PN" "2946-2601-3102-ND"
+			(at 35.56 34.29 0)
+			(effects
+				(font
+					(size 1.27 1.27)
+				)
+				(hide yes)
+			)
+		)
 		(pin "1"
 		)
@@
 			)
 		)
+		(property "DigiKey_PN" "2019-RK73H1JTTD1002FCT-ND"
+			(at 26.67 156.21 0)
+			(effects
+				(font
+					(size 1.27 1.27)
+				)
+				(hide yes)
+			)
+		)
 		(pin "1"
 		)
@@
 			)
 		)
+		(property "DigiKey_PN" "296-27898-1-ND"
+			(at 251.46 114.3 0)
+			(effects
+				(font
+					(size 1.27 1.27)
+				)
+				(hide yes)
+			)
+		)
 		(pin "1"
 		)
@@
 			)
 		)
+		(property "DigiKey_PN" "2019-RK73H1JTTD1002FCT-ND"
+			(at 26.67 167.64 0)
+			(effects
+				(font
+					(size 1.27 1.27)
+				)
+				(hide yes)
+			)
+		)
 		(pin "1"
 		)
@@
 			)
 		)
+		(property "DigiKey_PN" "2019-RK73H1JTTD5601FCT-ND"
+			(at 81.28 33.02 0)
+			(effects
+				(font
+					(size 1.27 1.27)
+				)
+				(hide yes)
+			)
+		)
 		(pin "1"
 		)
@@
 			)
 		)
+		(property "DigiKey_PN" "2019-RK73H1JTTD10R0FCT-ND"
+			(at 228.6 99.06 0)
+			(effects
+				(font
+					(size 1.27 1.27)
+				)
+				(hide yes)
+			)
+		)
 		(pin "1"
 		)
@@
 			)
 		)
+		(property "DigiKey_PN" "296-27898-1-ND"
+			(at 236.22 49.53 0)
+			(effects
+				(font
+					(size 1.27 1.27)
+				)
+				(hide yes)
+			)
+		)
 		(pin "1"
 		)
@@
 			)
 		)
+		(property "DigiKey_PN" "296-TPS2116DRLRCT-ND"
+			(at 139.7 104.14 0)
+			(effects
+				(font
+					(size 1.27 1.27)
+				)
+				(hide yes)
+			)
+		)
 		(pin "2"
 		)
@@
 			)
 		)
-		(property "Datasheet" "https://www.digikey.jp/short/3ww5zf50"
+		(property "Datasheet" "https://www.digikey.jp/short/58tn8j9t"
 			(at 158.75 104.14 90)
 			(effects
@@
 			)
 		)
+		(property "DigiKey_PN" "160-1434-1-ND"
+			(at 158.75 104.14 90)
+			(effects
+				(font
+					(size 1.27 1.27)
+				)
+				(hide yes)
+			)
+		)
 		(pin "1"
 		)
@@
 			)
 		)
+		(property "DigiKey_PN" "2019-RK73H1JTTD1002FCT-ND"
+			(at 106.68 55.88 90)
+			(effects
+				(font
+					(size 1.27 1.27)
+				)
+				(hide yes)
+			)
+		)
 		(pin "1"
 		)
@@
 			)
 		)
+		(property "DigiKey_PN" "2946-2601-3102-ND"
+			(at 34.29 63.5 0)
+			(effects
+				(font
+					(size 1.27 1.27)
+				)
+				(hide yes)
+			)
+		)
 		(pin "1"
 		)
@@
 			)
 		)
+		(property "DigiKey_PN" "2019-RK73H1JTTD1000FCT-ND"
+			(at 153.67 109.22 90)
+			(effects
+				(font
+					(size 1.27 1.27)
+				)
+				(hide yes)
+			)
+		)
 		(pin "1"
 		)
@@
 			)
 		)
-		(property "Akiduki_PN" ""
+		(property "Akiduki_PN" "111878"
 			(at 233.68 91.44 0)
 			(effects
@@
 			)
 		)
+		(property "DigiKey_PN" ""
+			(at 233.68 91.44 90)
+			(effects
+				(font
+					(size 1.27 1.27)
+				)
+				(hide yes)
+			)
+		)
 		(pin "1"
 		)
@@
 			)
 		)
+		(property "DigiKey_PN" "2019-RK73H1JTTD3483FCT-ND"
+			(at 107.95 104.14 0)
+			(effects
+				(font
+					(size 1.27 1.27)
+				)
+				(hide yes)
+			)
+		)
 		(pin "1"
 		)
@@
 			)
 		)
+		(property "DigiKey_PN" ""
+			(at 218.44 25.4 90)
+			(effects
+				(font
+					(size 1.27 1.27)
+				)
+				(hide yes)
+			)
+		)
+		(property "Akiduki_PN" "111878"
+			(at 218.44 25.4 90)
+			(effects
+				(font
+					(size 1.27 1.27)
+				)
+				(hide yes)
+			)
+		)
 		(pin "1"
 		)
@@
 			)
 		)
+		(property "DigiKey_PN" "2946-2601-3102-ND"
+			(at 34.29 71.12 0)
+			(effects
+				(font
+					(size 1.27 1.27)
+				)
+				(hide yes)
+			)
+		)
 		(pin "1"
 		)
@@
 			)
 		)
+		(property "DigiKey_PN" "2019-RK73H1JTTD10R0FCT-ND"
+			(at 223.52 34.29 0)
+			(effects
+				(font
+					(size 1.27 1.27)
+				)
+				(hide yes)
+			)
+		)
 		(pin "1"
 		)
@@
 			)
 		)
+		(property "DigiKey_PN" "2019-RK73H1JTTD10R0FCT-ND"
+			(at 213.36 34.29 0)
+			(effects
+				(font
+					(size 1.27 1.27)
+				)
+				(hide yes)
+			)
+		)
 		(pin "1"
 		)
@@
 			)
 		)
+		(property "DigiKey_PN" "2019-RK73H1JTTD3301FCT-ND"
+			(at 91.44 43.18 0)
+			(effects
+				(font
+					(size 1.27 1.27)
+				)
+				(hide yes)
+			)
+		)
 		(pin "1"
 		)
@@
 			)
 		)
+		(property "DigiKey_PN" "2019-RK73H1JTTD1003FCT-ND"
+			(at 107.95 111.76 0)
+			(effects
+				(font
+					(size 1.27 1.27)
+				)
+				(hide yes)
+			)
+		)
 		(pin "1"
 		)
@@
 			)
 		)
+		(property "DigiKey_PN" "2019-RK73H1JTTD10R0FCT-ND"
+			(at 238.76 99.06 0)
+			(effects
+				(font
+					(size 1.27 1.27)
+				)
+				(hide yes)
+			)
+		)
 		(pin "1"
 		)
@@
 			(at 101.6 60.96 0)
 			(effects
+				(font
+					(size 1.27 1.27)
+				)
+				(hide yes)
+			)
+		)
+		(property "DigiKey_PN" "2019-RK73H1JTTD1002FCT-ND"
+			(at 101.6 60.96 0)
+			(effects
