File: KiCad/LaunchController2.0/Switch.kicad_sch (KiCad schematic)
At the start: 32 parts, among them SW1 SW_Push, SW10 SW_Push, SW11 SW_Push, SW12 SW_Push, SW13 SW_Push, SW14 SW_Push, SW15 SW_Push, SW16 SW_Push, SW17 SW_Push, SW2 SW_Push, SW3 SW_Push, SW4 SW_Push, SW5 SW_Push, SW6 SW_Push, SW7 SW_Push, SW8 SW_Push, SW9 SW_Push

Commit message: シルクなどを調整
Parts:
- R14: renamed from R15; Digikey_PN (none) -> 2019-RK73H1JTTD1001FCT-ND
- R15: renamed from R16; Digikey_PN (none) -> 2019-RK73H1JTTD1001FCT-ND
- R16: renamed from R17; Digikey_PN (none) -> 2019-RK73H1JTTD1001FCT-ND
- R17: renamed from R18; Digikey_PN (none) -> 2019-RK73H1JTTD1001FCT-ND
- R18: renamed from R19; Digikey_PN (none) -> 2019-RK73H1JTTD1001FCT-ND
- R19: renamed from R20; Digikey_PN (none) -> 2019-RK73H1JTTD1001FCT-ND
- R20: renamed from R21; Digikey_PN (none) -> 2019-RK73H1JTTD1001FCT-ND
- R21: renamed from R22; Digikey_PN (none) -> 2019-RK73H1JTTD1001FCT-ND
- R22: renamed from R23; Digikey_PN (none) -> 2019-RK73H1JTTD1001FCT-ND
- R23: renamed from R24; Digikey_PN (none) -> 2019-RK73H1JTTD1001FCT-ND
- R24: renamed from R25; Digikey_PN (none) -> 2019-RK73H1JTTD1001FCT-ND
- R25: renamed from R26; Digikey_PN (none) -> 2019-RK73H1JTTD1001FCT-ND
- R26: renamed from R27; Digikey_PN (none) -> 2019-RK73H1JTTD1001FCT-ND
- R27: renamed from R28; Digikey_PN (none) -> 2019-RK73H1JTTD1001FCT-ND
- R28: renamed from R29; Digikey_PN (none) -> 2019-RK73H1JTTD1001FCT-ND
- SW1, SW2, SW3: Akiduki_PN (none) -> 106185
- SW10, SW11, SW12, SW13, SW14, SW15, SW16, SW17, SW4, SW5, SW6, SW7, SW8, SW9: Akiduki_PN (none) -> 108593
Other:
- company: (none) -> Tokai Student Rocket Project
- title: (none) -> Gen6 GSE Launch Controller 2.0

Commit message: とりあえずプッシュ
Parts:
- R14, R15, R16, R17, R18, R19, R20, R21, R22, R23, R24, R25, R26, R27, R28: DigiKey_PN (none) -> 2019-RK73H1JTTD1001FCT-ND
Changed lines of the file:
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@@
 			)
 		)
+		(property "DigiKey_PN" "2019-RK73H1JTTD1001FCT-ND"
+			(at 259.08 105.41 90)
+			(effects
+				(font
+					(size 1.27 1.27)
+				)
+				(hide yes)
+			)
+		)
 		(pin "1"
 		)
@@
 			)
 		)
+		(property "DigiKey_PN" "2019-RK73H1JTTD1001FCT-ND"
+			(at 171.45 86.36 90)
+			(effects
+				(font
+					(size 1.27 1.27)
+				)
+				(hide yes)
+			)
+		)
 		(pin "1"
 		)
@@
 			)
 		)
+		(property "DigiKey_PN" "2019-RK73H1JTTD1001FCT-ND"
+			(at 259.08 86.36 90)
+			(effects
+				(font
+					(size 1.27 1.27)
+				)
+				(hide yes)
+			)
+		)
 		(pin "1"
 		)
@@
 			)
 		)
+		(property "DigiKey_PN" "2019-RK73H1JTTD1001FCT-ND"
+			(at 259.08 48.26 90)
+			(effects
+				(font
+					(size 1.27 1.27)
+				)
+				(hide yes)
+			)
+		)
 		(pin "1"
 		)
@@
 			)
 		)
+		(property "DigiKey_PN" "2019-RK73H1JTTD1001FCT-ND"
+			(at 171.45 48.26 90)
+			(effects
+				(font
+					(size 1.27 1.27)
+				)
+				(hide yes)
+			)
+		)
 		(pin "1"
 		)
@@
 			)
 		)
+		(property "DigiKey_PN" "2019-RK73H1JTTD1001FCT-ND"
+			(at 171.45 29.21 90)
+			(effects
+				(font
+					(size 1.27 1.27)
+				)
+				(hide yes)
+			)
+		)
 		(pin "1"
 		)
@@
 			)
 		)
+		(property "DigiKey_PN" "2019-RK73H1JTTD1001FCT-ND"
+			(at 171.45 67.31 90)
+			(effects
+				(font
+					(size 1.27 1.27)
+				)
+				(hide yes)
+			)
+		)
 		(pin "1"
 		)
@@
 			)
 		)
+		(property "DigiKey_PN" "2019-RK73H1JTTD1001FCT-ND"
+			(at 259.08 124.46 90)
+			(effects
+				(font
+					(size 1.27 1.27)
+				)
+				(hide yes)
+			)
+		)
 		(pin "1"
 		)
@@
 			)
 		)
+		(property "DigiKey_PN" "2019-RK73H1JTTD1001FCT-ND"
+			(at 171.45 124.46 90)
+			(effects
+				(font
+					(size 1.27 1.27)
+				)
+				(hide yes)
+			)
+		)
 		(pin "1"
 		)
@@
 			)
 		)
+		(property "DigiKey_PN" "2019-RK73H1JTTD1001FCT-ND"
+			(at 259.08 67.31 90)
+			(effects
+				(font
+					(size 1.27 1.27)
+				)
+				(hide yes)
+			)
+		)
 		(pin "1"
 		)
@@
 			)
 		)
+		(property "DigiKey_PN" "2019-RK73H1JTTD1001FCT-ND"
+			(at 259.08 29.21 90)
+			(effects
+				(font
+					(size 1.27 1.27)
+				)
+				(hide yes)
+			)
+		)
 		(pin "1"
 		)
@@
 			)
 		)
+		(property "DigiKey_PN" "2019-RK73H1JTTD1001FCT-ND"
+			(at 259.08 162.56 90)
+			(effects
+				(font
+					(size 1.27 1.27)
+				)
+				(hide yes)
+			)
+		)
 		(pin "1"
 		)
@@
 			)
 		)
+		(property "DigiKey_PN" "2019-RK73H1JTTD1001FCT-ND"
+			(at 259.08 143.51 90)
+			(effects
+				(font
+					(size 1.27 1.27)
+				)
+				(hide yes)
+			)
+		)
 		(pin "1"
 		)
@@
 			)
 		)
+		(property "DigiKey_PN" "2019-RK73H1JTTD1001FCT-ND"
+			(at 71.12 55.88 90)
+			(effects
+				(font
+					(size 1.27 1.27)
+				)
+				(hide yes)
+			)
+		)
 		(pin "1"
 		)
@@
 			(at 171.45 105.41 90)
 			(effects
+				(font
+					(size 1.27 1.27)
+				)
+				(hide yes)
+			)
+		)
+		(property "DigiKey_PN" "2019-RK73H1JTTD1001FCT-ND"
+			(at 171.45 105.41 90)
+			(effects
