File: KiCad/SatelliteController2.0/SatelliteController2.0.kicad_sch (KiCad schematic)
At the start: 0 parts

Commit message: Build-1発行＆発注
Parts:
- added C1, C2: 15pF, Capacitor_SMD:C_0603_1608Metric_Pad1.08x0.95mm_HandSolder, symbol Device:C_Small
- added C10, C11, C3, C4, C5, C6, C7, C8: 0.1uF, Capacitor_SMD:C_0603_1608Metric_Pad1.08x0.95mm_HandSolder, symbol Device:C_Small
- added C9: 4.7uF, Capacitor_SMD:C_0603_1608Metric_Pad1.08x0.95mm_HandSolder, symbol Device:C_Small
- added D1: GS1010FL, Diode_SMD:D_SOD-123F, symbol Device:D_Small
- added D2: LED_O, LED_SMD:LED_0603_1608Metric_Pad1.05x0.95mm_HandSolder, symbol Device:LED_Small
- added F1: MF-NSMF050, Fuse:Fuse_1206_3216Metric_Pad1.42x1.75mm_HandSolder, symbol Device:Polyfuse_Small
- added H1, H2, H3, H4: MountingHole, MountingHole:MountingHole_4mm, symbol Mechanical:MountingHole
- added J1: CONN_ICSP, Connector_PinHeader_2.54mm:PinHeader_1x06_P2.54mm_Vertical, symbol Connector_Generic:Conn_01x06
- added J2: CONN_USB, TerminalBlock_WAGO:TerminalBlock_WAGO_2601-3104_1x04_P3.50mm_Vertical, symbol Connector_Generic:Conn_01x04
- added J3: USB_C_Receptacle_USB2.0_16P, Connector_USB:USB_C_Receptacle_GCT_USB4105-xx-A_16P_TopMnt_Horizontal, symbol Connector:USB_C_Receptacle_USB2.0_16P
- added L1: 10uH, Inductor_SMD:L_1210_3225Metric_Pad1.42x2.65mm_HandSolder, symbol Device:L
- added R1, R5, R7, R8: 10kR, Resistor_SMD:R_0603_1608Metric_Pad0.98x0.95mm_HandSolder, symbol Device:R_Small
- added R10, R11: 5.1kR, Resistor_SMD:R_0603_1608Metric_Pad0.98x0.95mm_HandSolder, symbol Device:R_Small
- added R12, R3, R4, R6: 1kR, Resistor_SMD:R_0603_1608Metric_Pad0.98x0.95mm_HandSolder, symbol Device:R_Small
- added R2, R9: 1MR, Resistor_SMD:R_0603_1608Metric_Pad0.98x0.95mm_HandSolder, symbol Device:R_Small
- added U1: ATMEGA2560-16AUR, Package_QFP:TQFP-100_14x14mm_P0.5mm, symbol MCU_Microchip_ATmega:ATmega2560-16A
- added U2: FT232RNL, Package_SO:SSOP-28_5.3x10.2mm_P0.65mm, symbol Interface_USB:FT232RL
- added U3: USBLC6-2SC6, Package_TO_SOT_SMD:SOT-23-6, symbol Power_Protection:USBLC6-2SC6
- added Y1: HUSG-16.000-20, Crystal:Crystal_HC49-4H_Vertical, symbol Device:Crystal_Small
Connections:
- new net: C2.1, R2.2, U1.33 (XTAL2), Y1.1
- new net: C8.2, U2.17 (3V3OUT)
- new net: C1.2, R2.1, U1.34 (XTAL1), Y1.2
- new net: J3.A5 (CC1), R10.1
- new net: C3.2, U1.98 (AREF)
- new net: J3.A7 (D-), J3.B7 (D-), U3.1 (I/O1)
- new net: J3.A6 (D+), J3.B6 (D+), U3.3 (I/O2)
- new net: R4.2, U1.3 (PE1)
- new net: R3.1, U1.2 (PE0)
- new net: C11.1, R12.1, U2.2 (DTR)
- new net: C7.1, L1.1, U1.100 (AVCC)
- new net: D2.2 (A), U1.26 (PB7)
- new net: F1.1, J3.A4 (VBUS), J3.A9 (VBUS), J3.B4 (VBUS), J3.B9 (VBUS)
- new net: J3.B5 (CC2), R11.1
- new net: D2.1 (K), R6.1
- new net +5V: C10.2, C4.1, C5.1, C6.1, D1.1 (K), J1.5 (Pin_5), L1.2, R1.1, R5.1, R7.1, R8.1, U1.10 (VCC), U1.31 (VCC), U1.61 (VCC), U1.80 (VCC), U2.20 (VCC), U2.4 (VCCIO)
- new net 7SEG_CLK: U1.89 (PK0)
- new net 7SEG_DIO: U1.88 (PK1)
- new net ALERT/RDY: U1.40 (PL5)
- new net CS_ADC: R5.2, U1.58 (PC5)
- new net CTL_CHECK: U1.54 (PC1)
- new net CTL_CLOSE: U1.53 (PC0)
- new net CTL_DUMP: U1.49 (PD6)
- new net CTL_FILL: U1.50 (PD7)
- new net CTL_IGNITOR: U1.48 (PD5)
- new net CTL_KILL: U1.64 (PJ1)
- new net CTL_O2: U1.51 (PG0)
- new net CTL_OPEN: U1.52 (PG1)
- new net CTL_POWER: U1.92 (PF5)
- new net CTL_PURGE: U1.55 (PC2)
- new net CTL_RESET: C11.2, D1.2 (A), J1.2 (Pin_2), R1.2, U1.30 (~{RESET})
- new net CTL_RS485_DERE: U1.56 (PC3)
- new net CTL_SAFETY: U1.27 (PH7)
- new net CTL_SHIFT: U1.47 (PD4)
- new net FLIGHT_MODE: U1.42 (PL7)
- new net GND: C1.1, C10.1, C2.2, C3.1, C4.2, C5.2, C6.2, C7.2, C8.1, C9.1, J1.1 (Pin_1), J2.1 (Pin_1), J3.A1 (GND), J3.A12 (GND), J3.B1 (GND), J3.B12 (GND), R10.2, R11.2, R12.2, R6.2, R9.2, U1.11 (GND), U1.32 (GND), U1.62 (GND), U1.81 (GND), U1.99 (GND), U2.18 (GND), U2.21 (GND), U2.25 (AGND), U2.26 (TEST), U2.7 (GND)
- new net GNDPWR: C9.2, J3.S1 (SHIELD), R9.1, U3.2 (GND)
- new net I2C_SCL: R7.2, U1.43 (PD0)
- new net I2C_SDA: R8.2, U1.44 (PD1)
- new net LED_CHECK: U1.25 (PB6)
- new net LED_COM: U1.84 (PK5)
- new net LED_ERROR: U1.83 (PK6)
- new net LED_FB_CLOSE: U1.23 (PB4)
- new net LED_FB_DUMP: U1.24 (PB5)
- new net LED_FB_FILL: U1.19 (PB0)
- new net LED_FB_IGNITOR: U1.16 (PH4)
- new net LED_FB_O2: U1.12 (PH0)
- new net LED_FB_OPEN: U1.18 (PH6)
- new net LED_FB_PURGE: U1.13 (PH1)
- new net LED_FB_SHIFT: U1.17 (PH5)
- new net LED_LOW_VOLTAGE: U1.82 (PK7)
- new net LED_POWER: U1.1 (PG5)
- new net LED_RS485_ACCESS: U1.57 (PC4)
- new net LED_SAFTEY: U1.28 (PG3)
- new net LED_TASK: U1.85 (PK4)
- new net LED_USB_ACCESS: U2.22 (CBUS1), U2.23 (CBUS0)
- new net SPI_MISO: J1.6 (Pin_6), U1.22 (PB3)
- new net SPI_MOSI: J1.3 (Pin_3), U1.21 (PB2)
- new net SPI_SCK: J1.4 (Pin_4), U1.20 (PB1)
- new net SW_CHECK: U1.29 (PG4)
- new net UART0_RX: R3.2, U2.1 (TXD)
- new net UART0_TX: R4.1, U2.5 (RXD)
- new net UART1_RX: U1.45 (PD2)
- new net UART1_TX: U1.46 (PD3)
- new net USB_D+: J2.2 (Pin_2), U2.15 (USBD+), U3.6 (I/O1)
- new net USB_D-: J2.3 (Pin_3), U2.16 (USBD-), U3.4 (I/O2)
- new net USB_VBUS: F1.2, J2.4 (Pin_4), U3.5 (VBUS)
- new net VALVE_MODE: U1.41 (PL6)
- new net VREF_N2O_PRESS: U1.87 (PK2)
- new net VREF_THERMISTOR: U1.93 (PF4)
- no-connect marks 0 -> 46
Other:
- added sheet Extension (Extension.kicad_sch)
- added sheet Indicator (Indicator.kicad_sch)
- added sheet Periferal (Periferal.kicad_sch)
- added sheet Power (Power.kicad_sch)
- added sheet Relay (Relay.kicad_sch)
- added sheet Switch (Switch.kicad_sch)
- note added: "48 FILL↔52 DUMP"
- note added: "50 IGN↔47 SHIFT"
- note added: "53 PURGE↔58 CHECK"
- note added: "CONNECTION ICSP"
- note added: "CONNECTION USB"
- note added: "Satellite Controller との変更点"
- note added: "USB-Serial"
- title: (none) -> Gen6 GSE Satellite Controller 2.0
