File: KiCad/SatelliteController2.0/SatelliteController2.0.kicad_sch (KiCad schematic)
At the start: 38 parts, among them J1 CONN_ICSP, J2 CONN_USB, J3 USB_C_Receptacle_USB2.0_16P, U1 ATMEGA2560-16AUR, U2 FT232RNL, U3 USBLC6-2SC6, Y1 HUSG-16.000-20

Commit message: シルクなどを調整
Parts:
- added S1: SLDR PASTE NO-CLN SAC305 50G, symbol Device:R
- C1, C2: Digikey_PN (none) -> 490-4941-1-ND
- C10, C11, C3, C4, C5, C6, C7, C8: Digikey_PN (none) -> 490-8020-1-ND
- C9: value 4.7uF -> 10nF; footprint Capacitor_SMD:C_0603_1608Metric_Pad1.08x0.95mm_HandSolder -> Capacitor_SMD:C_0805_2012Metric_Pad1.18x1.45mm_HandSolder; Digikey_PN (none) -> 490-GCM21B5C2E103FX0ALCT-ND
- D1: Akiduki_PN (none) -> 106014
- D2: Digikey_PN (none) -> SML-D12D8WT86CCT-ND
- F1: Akiduki_PN (none) -> 115300
- J1: Akiduki_PN (none) -> 101669
- J2: Digikey_PN (none) -> 2946-2601-3104-ND
- J3: Akiduki_PN (none) -> 114356
- L1: Akiduki_PN (none) -> 114977
- R1, R5, R7, R8: Digikey_PN (none) -> 2019-RK73H1JTTD1002FCT-ND
- R10, R11: Digikey_PN (none) -> 2019-RK73H1JTTD5101FCT-ND
- R12, R3, R4, R6: Digikey_PN (none) -> 2019-RK73H1JTTD1001FCT-ND
- R2: Digikey_PN (none) -> 2019-RK73H2BTTD1004FCT-ND
- R9: footprint Resistor_SMD:R_0603_1608Metric_Pad0.98x0.95mm_HandSolder -> Resistor_SMD:R_1206_3216Metric_Pad1.30x1.75mm_HandSolder; Digikey_PN (none) -> 2019-RK73H2BTTD1004FCT-ND
- U1: Akiduki_PN (none) -> 116567
- U2: Akiduki_PN (none) -> 118243
- U3: Digikey_PN (none) -> 497-5235-1-ND
- Y1: Akiduki_PN (none) -> 108671
Connections:
- net GND: now also U3.2 (GND)
- net GNDPWR: no longer U3.2 (GND)
- net USB_D+: now also U3.4 (I/O2); no longer U3.6 (I/O1)
- net USB_D-: now also U3.6 (I/O1); no longer U3.4 (I/O2)
- net LED_USB_ACCESS renamed LED_USB_RXLED
- net LED_USB_RXLED: no longer U2.23 (CBUS0)
- new net LED_USB_TXLED: U2.23 (CBUS0)
Other:
- note added: "BOM用"
- company: (none) -> Tokai Student Rocket Project

Commit message: BOM作成
Parts:
- C1, C2: Akiduki_PN (none) -> 113312; Digikey_PN 490-4941-1-ND -> (none)
- C10, C11, C3, C4, C5, C6, C7, C8: Akiduki_PN (none) -> 114559; Digikey_PN 490-8020-1-ND -> (none)
- D2: Digikey_PN SML-D12D8WT86CCT-ND -> SML-D15DWT86CCT-ND
- H1, H2, H3, H4: footprint MountingHole:MountingHole_4mm -> MountingHole:MountingHole_4.3mm_M4_Pad_Via
Changed lines of the file:
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@@
 			)
 		)
-		(property "Datasheet" "https://www.digikey.jp/short/4j7f3t3m"
+		(property "Datasheet" "https://akizukidenshi.com/catalog/g/g114559/"
 			(at 88.9 26.67 0)
 			(effects
@@
 			)
 		)
-		(property "Digikey_PN" "490-8020-1-ND "
+		(property "Digikey_PN" ""
+			(at 88.9 26.67 0)
+			(effects
+				(font
+					(size 1.27 1.27)
+				)
+				(hide yes)
+			)
+		)
+		(property "Akiduki_PN" "114559"
 			(at 88.9 26.67 0)
 			(effects
@@
 			)
 		)
-		(property "Datasheet" "https://akizukidenshi.com/catalog/g/gP-13312/"
+		(property "Datasheet" "https://akizukidenshi.com/catalog/g/g113312/"
 			(at 22.86 63.5 0)
 			(effects
@@
 			)
 		)
-		(property "Digikey_PN" "490-4941-1-ND "
+		(property "Digikey_PN" ""
+			(at 22.86 63.5 90)
+			(effects
+				(font
+					(size 1.27 1.27)
+				)
+				(hide yes)
+			)
+		)
+		(property "Akiduki_PN" "113312"
 			(at 22.86 63.5 90)
 			(effects
@@
 			)
 		)
-		(property "Datasheet" "https://www.digikey.jp/short/4j7f3t3m"
+		(property "Datasheet" "https://akizukidenshi.com/catalog/g/g114559/"
 			(at 99.06 26.67 0)
 			(effects
@@
 			)
 		)
-		(property "Digikey_PN" "490-8020-1-ND "
+		(property "Digikey_PN" ""
+			(at 99.06 26.67 0)
+			(effects
+				(font
+					(size 1.27 1.27)
+				)
+				(hide yes)
+			)
+		)
+		(property "Akiduki_PN" "114559"
 			(at 99.06 26.67 0)
 			(effects
@@
 			)
 		)
-		(property "Datasheet" "https://www.digikey.jp/short/4j7f3t3m"
+		(property "Datasheet" "https://akizukidenshi.com/catalog/g/g114559/"
 			(at 193.04 110.49 0)
 			(effects
@@
 			)
 		)
-		(property "Digikey_PN" "490-8020-1-ND "
+		(property "Digikey_PN" ""
+			(at 193.04 110.49 90)
+			(effects
+				(font
+					(size 1.27 1.27)
+				)
+				(hide yes)
+			)
+		)
+		(property "Akiduki_PN" "114559"
 			(at 193.04 110.49 90)
 			(effects
@@
 		(dnp no)
 		(fields_autoplaced yes)
-		(property "Reference" "#PWR018"
+		(property "Reference" "#PWR019"
 			(at 224.79 96.52 0)
 			(effects
@@
 			(project "SatelliteController2.0"
 				(path "/de793fd6-c32a-40e6-9ae3-03fbb6e83f09"
-					(reference "#PWR018")
+					(reference "#PWR019")
 					(unit 1)
 				)
@@
 			)
 		)
-		(property "Datasheet" "https://www.digikey.jp/short/4j7f3t3m"
+		(property "Datasheet" "https://akizukidenshi.com/catalog/g/g114559/"
 			(at 78.74 26.67 0)
 			(effects
@@
 			)
 		)
-		(property "Digikey_PN" "490-8020-1-ND "
+		(property "Digikey_PN" ""
+			(at 78.74 26.67 0)
+			(effects
+				(font
+					(size 1.27 1.27)
+				)
+				(hide yes)
+			)
+		)
+		(property "Akiduki_PN" "114559"
 			(at 78.74 26.67 0)
 			(effects
@@
 		(dnp no)
 		(fields_autoplaced yes)
-		(property "Reference" "#PWR019"
+		(property "Reference" "#PWR020"
 			(at 229.87 162.56 0)
 			(effects
@@
 			(project "SatelliteController2.0"
 				(path "/de793fd6-c32a-40e6-9ae3-03fbb6e83f09"
-					(reference "#PWR019")
+					(reference "#PWR020")
 					(unit 1)
 				)
@@
 			)
 		)
-		(property "Datasheet" "https://www.digikey.jp/short/4j7f3t3m"
+		(property "Datasheet" "https://akizukidenshi.com/catalog/g/g114559/"
 			(at 46.99 64.77 0)
 			(effects
@@
 			)
 		)
-		(property "Digikey_PN" "490-8020-1-ND "
+		(property "Digikey_PN" ""
+			(at 46.99 64.77 90)
+			(effects
+				(font
+					(size 1.27 1.27)
+				)
+				(hide yes)
+			)
+		)
+		(property "Akiduki_PN" "114559"
 			(at 46.99 64.77 90)
 			(effects
@@
 		(on_board yes)
 		(dnp no)
-		(property "Reference" "#PWR021"
+		(property "Reference" "#PWR023"
 			(at 260.35 134.62 0)
 			(effects
@@
 			(project "SatelliteController2.0"
 				(path "/de793fd6-c32a-40e6-9ae3-03fbb6e83f09"
-					(reference "#PWR021")
+					(reference "#PWR023")
 					(unit 1)
 				)
@@
 			)
 		)
-		(property "Footprint" "MountingHole:MountingHole_4mm"
+		(property "Footprint" "MountingHole:MountingHole_4.3mm_M4_Pad_Via"
 			(at 140.97 129.54 0)
 			(effects
@@
 			)
 		)
-		(property "Datasheet" "https://www.digikey.jp/short/4j7f3t3m"
+		(property "Datasheet" "https://akizukidenshi.com/catalog/g/g114559/"
 			(at 264.16 120.65 0)
 			(effects
@@
 			)
 		)
-		(property "Digikey_PN" "490-8020-1-ND "
+		(property "Digikey_PN" ""
+			(at 264.16 120.65 90)
+			(effects
+				(font
+					(size 1.27 1.27)
+				)
+				(hide yes)
+			)
+		)
+		(property "Akiduki_PN" "114559"
 			(at 264.16 120.65 90)
 			(effects
@@
 		(dnp no)
 		(fields_autoplaced yes)
-		(property "Reference" "#PWR0143"
+		(property "Reference" "#PWR018"
 			(at 220.98 85.09 0)
 			(effects
@@
 			(project "SatelliteController2.0"
 				(path "/de793fd6-c32a-40e6-9ae3-03fbb6e83f09"
-					(reference "#PWR0143")
+					(reference "#PWR018")
 					(unit 1)
 				)
@@
 			)
 		)
-		(property "Datasheet" "https://www.digikey.jp/short/4j7f3t3m"
+		(property "Datasheet" "https://akizukidenshi.com/catalog/g/g114559/"
 			(at 217.17 95.25 0)
 			(effects
@@
 			)
 		)
-		(property "Digikey_PN" "490-8020-1-ND "
+		(property "Digikey_PN" ""
+			(at 217.17 95.25 90)
+			(effects
+				(font
+					(size 1.27 1.27)
+				)
+				(hide yes)
+			)
+		)
+		(property "Akiduki_PN" "114559"
 			(at 217.17 95.25 90)
 			(effects
@@
 			)
 		)
-		(property "Footprint" "MountingHole:MountingHole_4mm"
+		(property "Footprint" "MountingHole:MountingHole_4.3mm_M4_Pad_Via"
 			(at 140.97 135.89 0)
 			(effects
@@
 			)
 		)
-		(property "Datasheet" "https://www.digikey.jp/short/4j7f3t3m"
+		(property "Datasheet" "https://akizukidenshi.com/catalog/g/g114559/"
 			(at 127 46.99 0)
 			(effects
@@
 			)
 		)
-		(property "Digikey_PN" "490-8020-1-ND "
+		(property "Digikey_PN" ""
+			(at 127 46.99 0)
+			(effects
+				(font
+					(size 1.27 1.27)
+				)
+				(hide yes)
+			)
+		)
+		(property "Akiduki_PN" "114559"
 			(at 127 46.99 0)
 			(effects
@@
 			)
 		)
-		(property "Footprint" "MountingHole:MountingHole_4mm"
+		(property "Footprint" "MountingHole:MountingHole_4.3mm_M4_Pad_Via"
 			(at 140.97 142.24 0)
 			(effects
@@
 			)
 		)
-		(property "Datasheet" "~"
+		(property "Datasheet" "https://www.digikey.jp/short/jprw48hq"
 			(at 17.78 190.5 0)
 			(effects
@@
 		(dnp no)
 		(fields_autoplaced yes)
-		(property "Reference" "#PWR0142"
+		(property "Reference" "#PWR022"
 			(at 260.35 57.15 0)
 			(effects
@@
 			(project "SatelliteController2.0"
 				(path "/de793fd6-c32a-40e6-9ae3-03fbb6e83f09"
-					(reference "#PWR0142")
+					(reference "#PWR022")
 					(unit 1)
 				)
@@
 		(dnp no)
 		(fields_autoplaced yes)
-		(property "Reference" "#PWR020"
+		(property "Reference" "#PWR021"
 			(at 250.19 72.39 0)
 			(effects
@@
 			(project "SatelliteController2.0"
 				(path "/de793fd6-c32a-40e6-9ae3-03fbb6e83f09"
-					(reference "#PWR020")
+					(reference "#PWR021")
 					(unit 1)
 				)
@@
 			)
 		)
-		(property "Footprint" "MountingHole:MountingHole_4mm"
+		(property "Footprint" "MountingHole:MountingHole_4.3mm_M4_Pad_Via"
 			(at 140.97 148.59 0)
 			(effects
@@
 			)
 		)
-		(property "Datasheet" ""
+		(property "Datasheet" "https://www.digikey.jp/short/3ww5zf50"
 			(at 128.27 90.17 90)
 			(effects
@@
 			)
 		)
-		(property "Digikey_PN" "SML-D12D8WT86CCT-ND "
+		(property "Digikey_PN" "SML-D15DWT86CCT-ND"
 			(at 128.27 90.17 0)
 			(effects
@@
 			)
 		)
-		(property "Datasheet" "https://akizukidenshi.com/catalog/g/gP-13312/"
+		(property "Datasheet" "https://akizukidenshi.com/catalog/g/g113312/"
 			(at 22.86 50.8 0)
 			(effects
@@
 			)
 		)
-		(property "Digikey_PN" "490-4941-1-ND "
+		(property "Digikey_PN" ""
+			(at 22.86 50.8 90)
+			(effects
+				(font
+					(size 1.27 1.27)
+				)
+				(hide yes)
+			)
+		)
+		(property "Akiduki_PN" "113312"
 			(at 22.86 50.8 90)
 			(effects

Commit message: とりあえずプッシュ
Parts:
- C9: DigiKey_PN (none) -> 490-GCM21B5C2E103FX0ALCT-ND
- D2: DigiKey_PN (none) -> 160-1434-1-ND
- J2: DigiKey_PN (none) -> 2946-2601-3104-ND
- R1, R5, R7, R8: DigiKey_PN (none) -> 2019-RK73H1JTTD1002FCT-ND
- R10, R11: DigiKey_PN (none) -> 2019-RK73H1JTTD5101FCT-ND
- R12, R3, R4, R6: DigiKey_PN (none) -> 2019-RK73H1JTTD1001FCT-ND
- R2, R9: DigiKey_PN (none) -> 2019-RK73H2BTTD1004FCT-ND
- S1: DigiKey_PN (none) -> SMD291SNL50T3-ND
- U3: DigiKey_PN (none) -> 497-5235-1-ND
