File: KiCad/SatelliteController2.0/SatelliteController2.0.kicad_pcb (KiCad board)
At the start: 2 copper layers, 150 x 100 mm, 222 parts, among them J1 CONN_ICSP, J10 CONN_ISOLATED_RS485_REPEATER, J11 CONN_UMBILICAL, J12 CONN_ISOLATED_RS485_REPEATER, J13 CONN_ISOLATED_RS485, J14 RELAY_POWER, J15 IGNITOR, J16 CONN_SORENOID_VALVE, J2 CONN_USB, J3 USB_C_Receptacle_USB2.0_16P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

Commit message: はんだ付けに使う資料を追加
Parts:
- D2: value LED_O -> LED_G
- moved C32 11.5 mm to (126.1, 128.4), turned to 180 degrees
- moved C33 11.5 mm to (115.7, 133.4), turned to 0 degrees
