File: KiCad/SatelliteController2.0/Extension.kicad_sch (KiCad schematic)
At the start: 2 parts, among them J7 CONN_STATUS_PANEL, J8 CONN_PANEL_BOARD_2

Commit message: シルクなどを調整
Parts:
- J7, J8: Digikey_PN (none) -> 2946-2601-3104-ND
Other:
- company: (none) -> Tokai Student Rocket Project
- title: (none) -> Gen6 GSE Satellite Controller 2.0

Commit message: とりあえずプッシュ
Parts:
- J7, J8: DigiKey_PN (none) -> 2946-2601-3104-ND
