File: KiCad/SatelliteController2.0/Periferal.kicad_sch (KiCad schematic)
At the start: 28 parts, among them J10 CONN_ISOLATED_RS485_REPEATER, J11 CONN_UMBILICAL, J12 CONN_ISOLATED_RS485_REPEATER, J13 CONN_ISOLATED_RS485, J9 CONN_N2O_PRESS, U10 TLP785F, U11 TLP785F, U8 ADS1115IDGS, U9 ADM2587E

Commit message: シルクなどを調整
Parts:
- added C31, C32: 470pF, Capacitor_SMD:C_1206_3216Metric_Pad1.33x1.80mm_HandSolder, symbol Device:C_Small
- C26, C27: value 0.1uF -> 10uF; footprint Capacitor_SMD:C_0603_1608Metric_Pad1.08x0.95mm_HandSolder -> Capacitor_SMD:C_0805_2012Metric_Pad1.18x1.45mm_HandSolder; Digikey_PN (none) -> 490-GCM21BC71C106KE36KCT-ND
- C28, C30: value 0.01uF -> 0.1uF; Digikey_PN (none) -> 490-8020-1-ND
- C29: Digikey_PN (none) -> 490-8020-1-ND
- C33: renamed from C31; value 0.1uF -> 10uF; footprint Capacitor_SMD:C_0603_1608Metric_Pad1.08x0.95mm_HandSolder -> Capacitor_SMD:C_0805_2012Metric_Pad1.18x1.45mm_HandSolder; Digikey_PN (none) -> 490-GCM21BC71C106KE36KCT-ND
- C34: renamed from C32; value 0.01uF -> 0.1uF; Digikey_PN (none) -> 490-8020-1-ND
- C35: renamed from C33; value 0.1uF -> 10uF; footprint Capacitor_SMD:C_0603_1608Metric_Pad1.08x0.95mm_HandSolder -> Capacitor_SMD:C_0805_2012Metric_Pad1.18x1.45mm_HandSolder; Digikey_PN (none) -> 490-GCM21BC71C106KE36KCT-ND
- C36: renamed from C34; value 0.01uF -> 0.1uF; Digikey_PN (none) -> 490-8020-1-ND
- D5, D6: Akiduki_PN (none) -> 106467
- FB1, FB2: Digikey_PN (none) -> 445-MMZ1608S202ATA00CT-ND
- J10, J11, J12, J13, J9: Digikey_PN (none) -> 2946-2601-3104-ND
- R27: renamed from R90; Digikey_PN (none) -> 2019-RK73H1JTTD1002FCT-ND
- R28: renamed from R27; Digikey_PN (none) -> 2019-RK73H1JTTD1002FCT-ND
- R29: renamed from R28; Akiduki_PN (none) -> 111795
- R30: renamed from R29; Digikey_PN (none) -> 2019-RK73H1JTTD1200FCT-ND
- R31: renamed from R30; Digikey_PN (none) -> 2019-RK73H1JTTD3000FCT-ND
- R32: renamed from R31; Digikey_PN (none) -> 2019-RK73H1JTTD3000FCT-ND
- U10, U11: Akiduki_PN (none) -> 107553
- U8: Digikey_PN (none) -> 296-38849-1-ND
- U9: Akiduki_PN (none) -> 113300
Connections:
- net GND: now also C31.1
- net GND2: now also C32.2
- new net: C31.2, C32.1
Other:
- company: (none) -> Tokai Student Rocket Project
- title: (none) -> Gen6 GSE Satellite Controller 2.0

Commit message: BOM作成
Parts:
- added R31: RS485_A, Resistor_SMD:R_0805_2012Metric_Pad1.20x1.40mm_HandSolder, symbol Device:R_Small
- added R32: RS485_B, Resistor_SMD:R_0805_2012Metric_Pad1.20x1.40mm_HandSolder, symbol Device:R_Small
- C26, C27, C33, C35: Akiduki_PN (none) -> 113388; Digikey_PN 490-GCM21BC71C106KE36KCT-ND -> (none)
- C28, C29, C30, C34, C36: Akiduki_PN (none) -> 114559; Digikey_PN 490-8020-1-ND -> (none)
- R30: footprint Resistor_SMD:R_0603_1608Metric_Pad0.98x0.95mm_HandSolder -> Resistor_SMD:R_0805_2012Metric_Pad1.20x1.40mm_HandSolder; Digikey_PN 2019-RK73H1JTTD1200FCT-ND -> 2019-RK73H2ATTD1200FCT-ND
- renumbered R31 to R33, R32 to R34
Connections:
- net at R30.1, U9.15 (Z), U9.17 (B): now also R32.1; no longer J10.3 (Pin_3), J12.3 (Pin_3), J13.3 (Pin_3)
- net at R30.2, U9.13 (Y), U9.18 (A): now also R31.1; no longer J10.2 (Pin_2), J12.2 (Pin_2), J13.2 (Pin_2)
- new net: J10.2 (Pin_2), J12.2 (Pin_2), J13.2 (Pin_2), R31.2
- new net: J10.3 (Pin_3), J12.3 (Pin_3), J13.3 (Pin_3), R32.2
Other:
- moved on the sheet: J10, J12

Commit message: とりあえずプッシュ
Parts:
- C31, C32: DigiKey_PN (none) -> 445-5785-1-ND
- FB1, FB2: DigiKey_PN (none) -> 445-MMZ1608S202ATA00CT-ND
- J10, J11, J12, J13, J9: DigiKey_PN (none) -> 2946-2601-3104-ND
- R27, R28: DigiKey_PN (none) -> 2019-RK73H1JTTD1002FCT-ND
- R30: DigiKey_PN (none) -> 2019-RK73H2ATTD1200FCT-ND
- R33, R34: DigiKey_PN (none) -> 2019-RK73H1JTTD3000FCT-ND
- U8: DigiKey_PN (none) -> 296-38849-1-ND
