File: KiCad/SatelliteController2.0/Power.kicad_sch (KiCad schematic)
At the start: 45 parts, among them J4 TO_CONVERTER, J5 FROM_CONVERTER, J6 DC_IN, Q1 TJ8S06M3L, Q2 2SC3325-Y, Q3 TJ8S06M3L, U4 TPS2116DRL, U5 NJM7805SDL1, U6 INA219BIDCNT, U7 INA219BIDCNT

Commit message: シルクなどを調整
Parts:
- C12, C16, C19, C23, C25: Digikey_PN (none) -> 490-8020-1-ND
- C13, C14: Digikey_PN (none) -> 490-GCM188D71H105KE36JCT-ND
- C15, C17: Akiduki_PN (none) -> 117338
- C18, C22, C24: Digikey_PN (none) -> 490-GCM21BC71C106KE36KCT-ND
- C20, C21: value uF -> 0.1uF; Digikey_PN (none) -> 490-8020-1-ND
- D3: Akiduki_PN (none) -> 106014
- D4: Digikey_PN (none) -> SML-D12Y8WT86CCT-ND
- J4, J5, J6: Digikey_PN (none) -> 2946-2601-3102-ND
- Q1, Q3: Akiduki_PN (none) -> 113964
- Q2: Akiduki_PN (none) -> 100628
- R13, R16, R17, TH1: Digikey_PN (none) -> 2019-RK73H1JTTD1002FCT-ND
- R14: Digikey_PN (none) -> 2019-RK73H1JTTD5601FCT-ND
- R15: Digikey_PN (none) -> 2019-RK73H1JTTD3301FCT-ND
- R18: value 348kR ±1% -> 348kR 1%; Digikey_PN (none) -> 2019-RK73H1JTTD3483FCT-ND
- R19: value 100kR ±1% -> 100kR 1%; Digikey_PN (none) -> 2019-RK73H1JTTD1003FCT-ND
- R20: Digikey_PN (none) -> 2019-RK73H1JTTD1000FCT-ND
- R21, R23, R24, R26: value 0R -> 10R; Digikey_PN (none) -> 2019-RK73H1JTTD10R0FCT-ND
- R22, R25: Digikey_PN (none) -> CRM2512-FX-R100ELFCT-ND
- TP1: footprint TestPoint:TestPoint_THTPad_D1.0mm_Drill0.5mm -> TestPoint:TestPoint_Keystone_5005-5009_Compact; Akiduki_PN (none) -> 116480
- TP2, TP3: footprint TestPoint:TestPoint_THTPad_D1.0mm_Drill0.5mm -> TestPoint:TestPoint_Keystone_5005-5009_Compact; Akiduki_PN (none) -> 116434
- TP4: footprint TestPoint:TestPoint_THTPad_D1.0mm_Drill0.5mm -> TestPoint:TestPoint_Keystone_5005-5009_Compact; Akiduki_PN (none) -> 116435
- U4: Digikey_PN (none) -> 296-TPS2116DRLRCT-ND
- U5: Akiduki_PN (none) -> 111237
- U6, U7: Digikey_PN (none) -> 296-27898-1-ND
Other:
- note added: "MULTIPLEXER"
- company: (none) -> Tokai Student Rocket Project
- title: (none) -> Gen6 GSE Satellite Controller 2.0

Commit message: BOM作成
Parts:
- C12, C16, C19, C20, C21, C23, C25: Akiduki_PN (none) -> 114559; Digikey_PN 490-8020-1-ND -> (none)
- C13, C14: Akiduki_PN (none) -> 130397; Digikey_PN 490-GCM188D71H105KE36JCT-ND -> (none)
- C18, C22, C24: Akiduki_PN (none) -> 113388; Digikey_PN 490-GCM21BC71C106KE36KCT-ND -> (none)
- D4: value LED_Y -> LED_O; Digikey_PN SML-D12Y8WT86CCT-ND -> SML-D15DWT86CCT-ND

Commit message: とりあえずプッシュ
Parts:
- D4: DigiKey_PN (none) -> 160-1434-1-ND
- J4, J5, J6: DigiKey_PN (none) -> 2946-2601-3102-ND
- R13, R16, R17, TH1: DigiKey_PN (none) -> 2019-RK73H1JTTD1002FCT-ND
- R14: DigiKey_PN (none) -> 2019-RK73H1JTTD5601FCT-ND
- R15: DigiKey_PN (none) -> 2019-RK73H1JTTD3301FCT-ND
- R18: DigiKey_PN (none) -> 2019-RK73H1JTTD3483FCT-ND
- R19: DigiKey_PN (none) -> 2019-RK73H1JTTD1003FCT-ND
- R20: DigiKey_PN (none) -> 2019-RK73H1JTTD1000FCT-ND
- R21, R23, R24, R26: DigiKey_PN (none) -> 2019-RK73H1JTTD10R0FCT-ND
- R22, R25: DigiKey_PN (none) -> CRM2512-FX-R100ELFCT-ND
- U4: DigiKey_PN (none) -> 296-TPS2116DRLRCT-ND
- U6, U7: DigiKey_PN (none) -> 296-27898-1-ND
