File: KiCad/SatelliteController2.0/Relay.kicad_sch (KiCad schematic)
At the start: 60 parts, among them J14 RELAY_POWER, J15 IGNITOR, J16 CONN_SORENOID_VALVE, Q10 AO3400A, Q11 AO3400A, Q12 AO3400A, Q13 AO3400A, Q4 AO3400A, Q5 AO3400A, Q6 AO3400A, Q7 AO3400A, Q8 AO3400A, Q9 AO3400A, U12 MCP3208

Commit message: シルクなどを調整
Parts:
- C37: renamed from C35; Digikey_PN (none) -> 490-8020-1-ND
- D27: renamed from D26; Akiduki_PN (none) -> 106014
- D28: renamed from D27; Akiduki_PN (none) -> 106014
- D29: renamed from D28; Akiduki_PN (none) -> 106014
- D30: renamed from D29; Akiduki_PN (none) -> 106014
- D31: renamed from D30; Akiduki_PN (none) -> 106014
- D32: renamed from D31; Akiduki_PN (none) -> 106014
- D33: renamed from D32; Akiduki_PN (none) -> 106014
- D34: renamed from D33; Akiduki_PN (none) -> 106014
- D35: renamed from D34; Akiduki_PN (none) -> 106014
- J14, J15: Digikey_PN (none) -> 2946-2601-3102-ND
- J16: Mouser_PN (none) -> 798-DF51A-8DP-2DSA
- Q10, Q11, Q12, Q13, Q4, Q5, Q6, Q7, Q8, Q9: Digikey_PN (none) -> 785-1000-1-ND
- R56: renamed from R54; Digikey_PN (none) -> 2019-RK73H1JTTD1200FCT-ND
- R57: renamed from R55; Digikey_PN (none) -> 2019-RK73H1JTTD1002FCT-ND
- R58: renamed from R56; Digikey_PN (none) -> 2019-RK73H1JTTD1200FCT-ND
- R59: renamed from R57; Digikey_PN (none) -> 2019-RK73H1JTTD1002FCT-ND
- R60: renamed from R58; Digikey_PN (none) -> 2019-RK73H1JTTD5602FCT-ND
- R61: renamed from R59; Digikey_PN (none) -> 2019-RK73H1JTTD3302FCT-ND
- R62: renamed from R60; Digikey_PN (none) -> 2019-RK73H1JTTD1200FCT-ND
- R63: renamed from R61; Digikey_PN (none) -> 2019-RK73H1JTTD1200FCT-ND
- R64: renamed from R62; Digikey_PN (none) -> 2019-RK73H1JTTD1002FCT-ND
- R65: renamed from R63; Digikey_PN (none) -> 2019-RK73H1JTTD1002FCT-ND
- R66: renamed from R64; Digikey_PN (none) -> 2019-RK73H1JTTD1200FCT-ND
- R67: renamed from R65; Digikey_PN (none) -> 2019-RK73H1JTTD1002FCT-ND
- R68: renamed from R66; Digikey_PN (none) -> 2019-RK73H1JTTD5602FCT-ND
- R69: renamed from R67; Digikey_PN (none) -> 2019-RK73H1JTTD3302FCT-ND
- R70: renamed from R68; Digikey_PN (none) -> 2019-RK73H1JTTD5602FCT-ND
- R71: renamed from R69; Digikey_PN (none) -> 2019-RK73H1JTTD3302FCT-ND
- R72: renamed from R70; Digikey_PN (none) -> 2019-RK73H1JTTD1200FCT-ND
- R73: renamed from R71; Digikey_PN (none) -> 2019-RK73H1JTTD1002FCT-ND
- R74: renamed from R72; Digikey_PN (none) -> 2019-RK73H1JTTD1200FCT-ND
- R75: renamed from R73; Digikey_PN (none) -> 2019-RK73H1JTTD1002FCT-ND
- R76: renamed from R74; Digikey_PN (none) -> 2019-RK73H1JTTD5602FCT-ND
- R77: renamed from R75; Digikey_PN (none) -> 2019-RK73H1JTTD3302FCT-ND
- R78: renamed from R76; Digikey_PN (none) -> 2019-RK73H1JTTD5602FCT-ND
- R79: renamed from R77; Digikey_PN (none) -> 2019-RK73H1JTTD3302FCT-ND
- R80: renamed from R78; Digikey_PN (none) -> 2019-RK73H1JTTD1200FCT-ND
- R81: renamed from R79; Digikey_PN (none) -> 2019-RK73H1JTTD1002FCT-ND
- R82: renamed from R80; Digikey_PN (none) -> 2019-RK73H1JTTD1200FCT-ND
- R83: renamed from R81; Digikey_PN (none) -> 2019-RK73H1JTTD1002FCT-ND
- R84: renamed from R82; Digikey_PN (none) -> 2019-RK73H1JTTD1200FCT-ND
- R85: renamed from R83; Digikey_PN (none) -> 2019-RK73H1JTTD1002FCT-ND
- R86: renamed from R84; Digikey_PN (none) -> 2019-RK73H1JTTD5602FCT-ND
- R87: renamed from R85; Digikey_PN (none) -> 2019-RK73H1JTTD3302FCT-ND
- R88: renamed from R86; Digikey_PN (none) -> 2019-RK73H1JTTD5602FCT-ND
- R89: renamed from R87; Digikey_PN (none) -> 2019-RK73H1JTTD3302FCT-ND
- R90: renamed from R88; Digikey_PN (none) -> 2019-RK73H1JTTD5602FCT-ND
- R91: renamed from R89; Digikey_PN (none) -> 2019-RK73H1JTTD3302FCT-ND
- U12: Akiduki_PN (none) -> 100238
Other:
- company: (none) -> Tokai Student Rocket Project
- title: (none) -> Gen6 GSE Satellite Controller 2.0

Commit message: BOM作成
Parts:
- C37: Akiduki_PN (none) -> 114559; Digikey_PN 490-8020-1-ND -> (none)
- renumbered R56 to R58, R57 to R59, R58 to R60, R59 to R61, R60 to R62, R61 to R63, R62 to R64, R63 to R65, R64 to R66, R65 to R67, R66 to R68, R67 to R69, R68 to R70, R69 to R71, R70 to R72, R71 to R73, R72 to R74, R73 to R75, R74 to R76, R75 to R77, R76 to R78, R77 to R79, R78 to R80, R79 to R81, R80 to R82, R81 to R83, R82 to R84, R83 to R85, R84 to R86, R85 to R87, R86 to R88, R87 to R89, R88 to R90, R89 to R91, R90 to R92, R91 to R93

Commit message: とりあえずプッシュ
Parts:
- J14, J15: DigiKey_PN (none) -> 2946-2601-3102-ND
- Q10, Q11, Q12, Q13, Q4, Q5, Q6, Q7, Q8, Q9: DigiKey_PN (none) -> 785-1000-1-ND
- R58, R60, R64, R65, R68, R74, R76, R82, R84, R86: DigiKey_PN (none) -> 2019-RK73H1JTTD1200FCT-ND
- R59, R61, R66, R67, R69, R75, R77, R83, R85, R87: DigiKey_PN (none) -> 2019-RK73H1JTTD1002FCT-ND
- R62, R70, R72, R78, R80, R88, R90, R92: DigiKey_PN (none) -> 2019-RK73H1JTTD5602FCT-ND
- R63, R71, R73, R79, R81, R89, R91, R93: DigiKey_PN (none) -> 2019-RK73H1JTTD3302FCT-ND
