File: KiCad/SatelliteController2.0/Switch.kicad_sch (KiCad schematic)
At the start: 8 parts, among them SW1 RUN_SW, SW2 KILL_SW, SW3 SAFETY_SW, SW4 RESET_SW, SW5 CHECK_SW

Commit message: シルクなどを調整
Parts:
- R53: renamed from R51; Digikey_PN (none) -> 2019-RK73H1JTTD1001FCT-ND
- R54: renamed from R52; Digikey_PN (none) -> 2019-RK73H1JTTD1001FCT-ND
- R55: renamed from R53; Digikey_PN (none) -> 2019-RK73H1JTTD1001FCT-ND
- SW1, SW2, SW4: Akiduki_PN (none) -> 106185
- SW3, SW5: Akiduki_PN (none) -> 108593
Other:
- company: (none) -> Tokai Student Rocket Project
- title: (none) -> Gen6 GSE Satellite Controller 2.0

Commit message: BOM作成
Parts:
- renumbered R53 to R55, R54 to R56, R55 to R57
Changed lines of the file:
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@@
 		(dnp no)
 		(fields_autoplaced yes)
-		(property "Reference" "#PWR0102"
+		(property "Reference" "#PWR0104"
 			(at 38.1 158.75 0)
 			(effects
@@
 			(project "SatelliteController2.0"
 				(path "/de793fd6-c32a-40e6-9ae3-03fbb6e83f09/fa9cd0b2-3ba5-4aff-8a78-22cf32cf071e"
-					(reference "#PWR0102")
+					(reference "#PWR0104")
 					(unit 1)
 				)
@@
 		(dnp no)
 		(fields_autoplaced yes)
-		(property "Reference" "#PWR0104"
+		(property "Reference" "#PWR0106"
 			(at 40.64 109.22 0)
 			(effects
@@
 			(project "SatelliteController2.0"
 				(path "/de793fd6-c32a-40e6-9ae3-03fbb6e83f09/fa9cd0b2-3ba5-4aff-8a78-22cf32cf071e"
-					(reference "#PWR0104")
+					(reference "#PWR0106")
 					(unit 1)
 				)
@@
 		(dnp no)
 		(fields_autoplaced yes)
-		(property "Reference" "R53"
+		(property "Reference" "R55"
 			(at 63.5 60.9599 0)
 			(effects
@@
 			(project ""
 				(path "/de793fd6-c32a-40e6-9ae3-03fbb6e83f09/fa9cd0b2-3ba5-4aff-8a78-22cf32cf071e"
-					(reference "R53")
+					(reference "R55")
 					(unit 1)
 				)
@@
 		(dnp no)
 		(fields_autoplaced yes)
-		(property "Reference" "#PWR0106"
+		(property "Reference" "#PWR0108"
 			(at 60.96 73.66 0)
 			(effects
@@
 			(project "SatelliteController2.0"
 				(path "/de793fd6-c32a-40e6-9ae3-03fbb6e83f09/fa9cd0b2-3ba5-4aff-8a78-22cf32cf071e"
-					(reference "#PWR0106")
+					(reference "#PWR0108")
 					(unit 1)
 				)
@@
 		(dnp no)
 		(fields_autoplaced yes)
-		(property "Reference" "#PWR0108"
+		(property "Reference" "#PWR0110"
 			(at 68.58 90.17 0)
 			(effects
@@
 			(project "SatelliteController2.0"
 				(path "/de793fd6-c32a-40e6-9ae3-03fbb6e83f09/fa9cd0b2-3ba5-4aff-8a78-22cf32cf071e"
-					(reference "#PWR0108")
+					(reference "#PWR0110")
 					(unit 1)
 				)
@@
 		(dnp no)
 		(fields_autoplaced yes)
-		(property "Reference" "#PWR0107"
+		(property "Reference" "#PWR0109"
 			(at 60.96 177.8 0)
 			(effects
@@
 			(project "SatelliteController2.0"
 				(path "/de793fd6-c32a-40e6-9ae3-03fbb6e83f09/fa9cd0b2-3ba5-4aff-8a78-22cf32cf071e"
-					(reference "#PWR0107")
+					(reference "#PWR0109")
 					(unit 1)
 				)
@@
 		(dnp no)
 		(fields_autoplaced yes)
-		(property "Reference" "#PWR0103"
+		(property "Reference" "#PWR0105"
 			(at 40.64 43.18 0)
 			(effects
@@
 			(project "SatelliteController2.0"
 				(path "/de793fd6-c32a-40e6-9ae3-03fbb6e83f09/fa9cd0b2-3ba5-4aff-8a78-22cf32cf071e"
-					(reference "#PWR0103")
+					(reference "#PWR0105")
 					(unit 1)
 				)
@@
 		(dnp no)
 		(fields_autoplaced yes)
-		(property "Reference" "R54"
+		(property "Reference" "R56"
 			(at 63.5 166.3699 0)
 			(effects
@@
 			(project ""
 				(path "/de793fd6-c32a-40e6-9ae3-03fbb6e83f09/fa9cd0b2-3ba5-4aff-8a78-22cf32cf071e"
-					(reference "R54")
+					(reference "R56")
 					(unit 1)
 				)
@@
 		(dnp no)
 		(fields_autoplaced yes)
-		(property "Reference" "#PWR0105"
+		(property "Reference" "#PWR0107"
 			(at 40.64 143.51 0)
 			(effects
@@
 			(project "SatelliteController2.0"
 				(path "/de793fd6-c32a-40e6-9ae3-03fbb6e83f09/fa9cd0b2-3ba5-4aff-8a78-22cf32cf071e"
-					(reference "#PWR0105")
+					(reference "#PWR0107")
 					(unit 1)
 				)
@@
 		(on_board yes)
 		(dnp no)
-		(property "Reference" "R55"
+		(property "Reference" "R57"
 			(at 63.5 83.82 90)
 			(effects
@@
 			(project "SatelliteController2.0"
 				(path "/de793fd6-c32a-40e6-9ae3-03fbb6e83f09/fa9cd0b2-3ba5-4aff-8a78-22cf32cf071e"
-					(reference "R55")
+					(reference "R57")
 					(unit 1)
 				)
@@
 		(dnp no)
 		(fields_autoplaced yes)
-		(property "Reference" "#PWR0101"
+		(property "Reference" "#PWR0103"
 			(at 38.1 58.42 0)
 			(effects
@@
 			(project "SatelliteController2.0"
 				(path "/de793fd6-c32a-40e6-9ae3-03fbb6e83f09/fa9cd0b2-3ba5-4aff-8a78-22cf32cf071e"
-					(reference "#PWR0101")
-					(unit 1)
-				)
+					(reference "#PWR0103")
+					(unit 1)
+				)

Commit message: とりあえずプッシュ
Parts:
- R55, R56, R57: DigiKey_PN (none) -> 2019-RK73H1JTTD1001FCT-ND
