File: KiCad/SatelliteNode/SatelliteNode-Switch.kicad_pcb (KiCad board)
At the start: 2 copper layers, 30 x 30 mm, 15 parts, among them J1 DF51A-4P-2DS, M3 MountingHole, Q1 DTC123EU3

Commit message: SatelliteNode Build-1を発行
Other:
- board text added: "NC"
- board text removed: "NO"
