File: KiCad/SatelliteNode/SatelliteNode-Switch.kicad_sch (KiCad schematic)
At the start: 11 parts, among them J1 DF51A-4P-2DS, Q1 DTC123EU3

Commit message: SatelliteNode Build-1を発行
Changed lines of the file:
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@@
 		)
 	)
-	(text "NO"
+	(text "NC"
 		(exclude_from_sim no)
 		(at 100.33 69.342 0)
