File: KiCad/SatelliteNode/SatelliteNode.kicad_sch (KiCad schematic)
At the start: 18 parts, among them J1 Conn_02x06_Counter_Clockwise, J2 Conn_01x04, J3 Conn_01x04, J4 Conn_01x04, J5 Conn_01x04, J6 Conn_01x04, J7 Conn_01x04, U1 XIAO-ESP32-C6, U2 NJM2845DL1-05, U3 74HC14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

Commit message: SatelliteNode-Switch Build-1発行
Parts:
- removed J1: Conn_02x06_Counter_Clockwise, symbol Connector_Generic:Conn_02x06_Counter_Clockwise
- added J1: Isolated_RS485, TSRP_IC:StrawberryLinux_ADM2582, symbol Connector_Generic:Conn_02x10_Odd_Even
- added J8: I2C_Connector, symbol Connector_Generic:Conn_01x04
- added J9: 12V_Connector, TSRP_Connector_Hirose:DF51-2P-2DS, symbol Connector_Generic:Conn_01x02
- C3: value C_Small -> 0.1uF
- D1: value D_Schottky_Small_Filled -> SS2040; footprint (none) -> Diode_SMD:D_SOD-123F
- U1: footprint Module:MOUDLE14P-XIAO-DIP-SMD -> TSRP_Seeed_XIAO:XIAO-ESP32-C6-DIP
- U3: footprint (none) -> Package_DIP:DIP-14_W7.62mm_LongPads
Connections:
- net +12V: now also J9.2 (Pin_2)
- net +3.3V: now also J1.10 (Pin_10), J8.2 (Pin_2)
- net GND: now also J1.9 (Pin_9), J8.1 (Pin_1), J9.1 (Pin_1)
- net I2C_SCL: now also J8.3 (Pin_3)
- net I2C_SDA: now also J8.4 (Pin_4)
- net RS485_DI: now also J1.5 (Pin_5)
- net RS485_RO: now also J1.3 (Pin_3)
- net RS485_~{RE}_DE: now also J1.15 (Pin_15), J1.17 (Pin_17)
- net SPI_MISO: now reaches U1.10 (GPIO20/D9/MISO)
- net SPI_MOSI: now reaches U1.11 (GPIO18/D10/MOSI)
- net SPI_SCK: now reaches U1.9 (GPIO19/D8/SCK)
- no-connect marks 2 -> 20
Other:
- note added: "SSD1306など"
- moved on the sheet: C1, C2, D1, D2, R1, R2, U1, U2

Commit message: SatelliteNode Build-1を発行
Parts:
- removed C2: 0.1uF, symbol Device:C_Small
- removed D1: SS2040, Diode_SMD:D_SOD-123F, symbol Device:D_Schottky_Small_Filled
- removed D2: 1N4148W, Diode_SMD:D_SOD-123, symbol Device:D_Small
- removed J8: I2C_Connector, symbol Connector_Generic:Conn_01x04
- removed U2: NJM2845DL1-05, Package_TO_SOT_SMD:TO-252-2, symbol Regulator_Linear:L7805
- added C4: 0.1uF, Capacitor_SMD:C_0603_1608Metric, symbol Device:C_Small
- added D1: BZX55C3V3, Diode_THT:D_DO-35_SOD27_P7.62mm_Horizontal, symbol Device:D_Zener_Small
- added D2: RB160M-30TR, TSRP_Diode:SOD-123FL_Handsolder, symbol Device:D_Schottky_Small
- added F1: MF-R050, Fuse:Fuse_Bourns_MF-RG300, symbol Device:Polyfuse_Small
- added H1, H2, H3: MountingHole, MountingHole:MountingHole_3.2mm_M3, symbol Mechanical:MountingHole
- added R3, R5: 10kR 1%, Resistor_SMD:R_0603_1608Metric, symbol Device:R_Small
- added U2: SSD1306, TSRP_IC:SSD1306, symbol TSRP_IC:SSD1306
- added U6: BP5293-50, Package_TO_SOT_THT:TO-220F-3_Vertical, symbol TSRP_IC:BP5293-50
- C1: value 2.2uF -> 0.1uF; footprint (none) -> Capacitor_SMD:C_0603_1608Metric
- C3: footprint (none) -> Capacitor_SMD:C_0603_1608Metric
- J1: renamed from J9; footprint TSRP_Connector_Hirose:DF51-2P-2DS -> TSRP_Connector_Hirose:DF51A-2P-2DSA
- J4: renamed from J3; footprint (none) -> TSRP_Connector_Hirose:DF51A-4P-2DSA
- J5: renamed from J4; footprint (none) -> TSRP_Connector_Hirose:DF51A-4P-2DSA
- J6: renamed from J5; footprint (none) -> TSRP_Connector_Hirose:DF51A-4P-2DSA
- J7: renamed from J6; footprint (none) -> TSRP_Connector_Hirose:DF51A-4P-2DSA
- J8: renamed from J7; footprint (none) -> TSRP_Connector_Hirose:DF51A-4P-2DSA
- R1, R2: value 10kR -> 4.7kR; footprint (none) -> Resistor_SMD:R_0603_1608Metric
- renumbered J1 to J2, J2 to J3, U1 to U3, U3 to U5
Connections:
- net +12V: now also F1.1
- net +3.3V: now also C4.1, U2.2 (VCC)
- net +5V: now also D2.2 (A), R3.1, U6.3 (VOUT); no longer C1.1
- net GND: now also C1.1, C4.2, D1.2 (A), R5.1, U2.1 (GND), U6.2 (GND); no longer C1.2
- net I2C_SCL: now also U2.3 (SCL)
- net I2C_SDA: now also U2.4 (SDA)
- net Switch_Out_0: now also U4.23 (GPA2), U5.1; no longer U4.21 (GPA0), U5.2
- net Switch_Out_1: now also U5.3; no longer U5.4
- net Switch_Out_2: now also U4.21 (GPA0), U5.5; no longer U4.23 (GPA2), U5.6
- net Switch_Out_3: now also U4.26 (GPA5), U5.9; no longer U4.24 (GPA3), U5.8
- net Switch_Out_4: now also U5.11; no longer U5.10
- net Switch_Out_5: now also U4.24 (GPA3), U5.13; no longer U4.26 (GPA5), U5.12
- net at J6.3 (Pin_3): now also U5.8; no longer U5.9
- net at J7.3 (Pin_3): now also U5.10; no longer U5.11
- net at U3.14 (VBUS): now also D2.1 (K)
- net 5V_ADC: now reaches U3.2 (GPIO1/A1/D1)
- net 5V_ADC: now also C1.2, D1.1 (K), R3.2, R5.2
- net at J8.3 (Pin_3): now also U5.12; no longer U5.13
- net at J5.3 (Pin_3): now also U5.6; no longer U5.5
- net at J3.3 (Pin_3): now also U5.2; no longer U5.1
- net at J4.3 (Pin_3): now also U5.4; no longer U5.3
- new net: F1.2, U6.1 (VIN)
- no-connect marks 20 -> 22
Other:
- note removed: "SSD1306など"
- moved on the sheet: J1, R1, R2

Commit message: Build-2 を発行
Parts:
- added R10, R4, R6, R7, R8, R9: 10kR, Resistor_SMD:R_0603_1608Metric, symbol Device:R_Small
Connections:
- net +3.3V: now also R10.1, R4.1, R6.1, R7.1, R8.1, R9.1
- net Switch_Out_0: now also U5.2; no longer U5.1
- net Switch_Out_1: now also U5.4; no longer U5.3
- net Switch_Out_2: now also U5.6; no longer U5.5
- net Switch_Out_3: now also U5.8; no longer U5.9
- net Switch_Out_4: now also U5.10; no longer U5.11
- net Switch_Out_5: now also U5.12; no longer U5.13
- net at J6.3 (Pin_3): now also U5.9, R8.2; no longer U5.8
- net at J7.3 (Pin_3): now also U5.11, R9.2; no longer U5.10
- net at J8.3 (Pin_3): now also U5.13, R10.2; no longer U5.12
- net at J5.3 (Pin_3): now also U5.5, R7.2; no longer U5.6
- net at J3.3 (Pin_3): now also U5.1, R4.2; no longer U5.2
- net at J4.3 (Pin_3): now also U5.3, R6.2; no longer U5.4
Other:
- moved on the sheet: J3, J4, J5, J6, J7, J8, U5A, U5B, U5C, U5D, U5E, U5F
