File: KiCad/StatusPanel/StatusPanel.kicad_sch (KiCad schematic)
At the start: 36 parts, among them J1 CONN, J10 CONN_12V_CTL, J11 CONN_12V_GND, J12 CONN_TASK_CTL, J13 CONN_TASK_GND, J14 CONN_5V_CTL, J15 CONN_5V_GND, J16 CONN_COM_CTL, J17 CONN_COM_GND, J18 CONN_LOW_CTL, J19 CONN_LOW_GND, J2 CONN_RESET_CTL, J20 CONN_ERROR_CTL, J21 CONN_ERROR_GND, J3 CONN_RESET_GND, J4 CONN_USB_5V, J5 CONN_USB_CTL, J6 CONN_INPUT_CTL, J7 CONN_INPUT_GND, J8 CONN_RS485_CTL, J9 CONN_RS485_GND, U1 2281SB, U2 TM1637

Commit message: 回路図を出力
Other:
- company: (none) -> Tokai Student Rocket Project
- title: (none) -> Gen6 GSE Statut Panel
